File: microcap/pcb/pcb.brd (EAGLE design)
At the start: 32 parts

Commit message: pcb design
Routing:
- net S$67: track 238.8 -> 236.6 mm
Changed lines of the file:
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@@
 <wire x1="-12.5" y1="47.5" x2="-15" y2="47.5" width="0.4064" layer="16"/>
 <wire x1="-15" y1="47.5" x2="-22.5" y2="55" width="0.4064" layer="16"/>
-<wire x1="75" y1="110" x2="-22.5" y2="110" width="0.4064" layer="16"/>
-<wire x1="-22.5" y1="110" x2="-22.5" y2="55" width="0.4064" layer="16"/>
+<wire x1="75" y1="110" x2="-18.75" y2="110" width="0.4064" layer="16"/>
+<wire x1="-22.5" y1="106.25" x2="-22.5" y2="55" width="0.4064" layer="16"/>
 <wire x1="75" y1="110" x2="80" y2="105" width="0.4064" layer="16"/>
 <wire x1="80" y1="105" x2="80" y2="91.25" width="0.4064" layer="16"/>
@@
 <wire x1="46.25" y1="91.25" x2="45" y2="91.25" width="0.4064" layer="16"/>
 <wire x1="45" y1="91.25" x2="42.5" y2="88.75" width="0.4064" layer="16"/>
+<wire x1="-22.5" y1="106.25" x2="-18.75" y2="110" width="0.4064" layer="16"/>
 </signal>
 <signal name="S$18">
