File: microcap/pcb/pcb_v2.brd (EAGLE design)
At the start: 98 parts

Commit message: pcb design
Parts:
- moved E$15 1.27 mm to (71.1, 48.3)
- moved E$43 1.27 mm to (71.1, 81.3)
Connections:
- new net S$12: E$17.A, E$18.C
- new net S$19: E$16.A, E$19.C
- new net S$22: E$45.A, E$46.C
- new net S$25: E$44.A, E$47.C
- net S$8: now also E$24.1, E$72.1
Routing:
- net S$8: track 260.2 -> 414.7 mm
- net S$25: track 0.00 -> 2.54 mm
- net S$22: track 0.00 -> 2.54 mm
- net S$19: track 0.00 -> 2.54 mm
- net S$12: track 0.00 -> 2.54 mm
- net S$3: track 18.3 -> 19.6 mm
- net S$2: track 20.1 -> 18.8 mm
- net S$16: track 20.1 -> 18.8 mm
- net S$13: track 18.3 -> 19.6 mm
- added copper zone on layer 16, net S$26
