File: microcap/pcb/pcb_v3.brd (EAGLE design)
At the start: 99 parts

Commit message: pcb pdf added
Parts:
- removed E$93: (no value), resistor:0207/10
Connections:
- removed net S$26: E$58.1, E$93.2
- net S$18: now also E$58.1, E$59.1; no longer E$93.1
Routing:
- net S$26: track 5.39 -> 0.00 mm
Changed lines of the file:
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@@
 <element name="E$99" library="pinhead" package="1X01" value="" x="110.49" y="82.55"/>
 <element name="E$100" library="pinhead" package="1X01" value="" x="110.49" y="80.01"/>
-<element name="E$93" library="resistor" package="0207/10" value="" x="78.74" y="91.44" rot="R90"/>
 </elements>
 <signals>
@@
 </signal>
 <signal name="S$18">
-<contactref element="E$50" pad="2"/>
-<contactref element="E$4" pad="C"/>
-<wire x1="73.66" y1="97.79" x2="74.93" y2="96.52" width="0.4064" layer="16"/>
-<wire x1="63.5" y1="92.71" x2="62.23" y2="92.71" width="0.4064" layer="16"/>
-<wire x1="62.23" y1="92.71" x2="60.96" y2="93.98" width="0.4064" layer="16"/>
-<wire x1="69.85" y1="97.79" x2="73.66" y2="97.79" width="0.4064" layer="16"/>
-<wire x1="69.85" y1="95.25" x2="69.85" y2="97.79" width="0.4064" layer="16"/>
-<contactref element="E$44" pad="C"/>
-<wire x1="60.96" y1="97.79" x2="69.85" y2="97.79" width="0.4064" layer="16"/>
-<wire x1="60.96" y1="93.98" x2="60.96" y2="97.79" width="0.4064" layer="16"/>
-<contactref element="E$45" pad="C"/>
-<wire x1="58.42" y1="97.79" x2="60.96" y2="97.79" width="0.4064" layer="16"/>
-<wire x1="58.42" y1="96.52" x2="58.42" y2="97.79" width="0.4064" layer="16"/>
-<wire x1="49.53" y1="92.71" x2="50.8" y2="92.71" width="0.4064" layer="16"/>
-<wire x1="50.8" y1="92.71" x2="52.07" y2="93.98" width="0.4064" layer="16"/>
-<wire x1="54.61" y1="97.79" x2="58.42" y2="97.79" width="0.4064" layer="16"/>
-<wire x1="54.61" y1="96.52" x2="54.61" y2="97.79" width="0.4064" layer="16"/>
-<contactref element="E$1" pad="C"/>
-<wire x1="52.07" y1="97.79" x2="54.61" y2="97.79" width="0.4064" layer="16"/>
-<wire x1="52.07" y1="93.98" x2="52.07" y2="97.79" width="0.4064" layer="16"/>
-<wire x1="43.18" y1="97.79" x2="52.07" y2="97.79" width="0.4064" layer="16"/>
-<wire x1="43.18" y1="95.25" x2="43.18" y2="97.79" width="0.4064" layer="16"/>
-<wire x1="39.37" y1="97.79" x2="43.18" y2="97.79" width="0.4064" layer="16"/>
-<wire x1="74.93" y1="96.52" x2="78.74" y2="92.71" width="0.4064" layer="16"/>
-<contactref element="E$93" pad="1"/>
-<wire x1="78.74" y1="92.71" x2="78.74" y2="86.36" width="0.4064" layer="16"/>
 <contactref element="E$70" pad="1"/>
-<wire x1="85.09" y1="85.09" x2="85.09" y2="49.53" width="0.4064" layer="16"/>
+<wire x1="85.09" y1="92.71" x2="85.09" y2="49.53" width="0.4064" layer="16"/>
 <wire x1="82.55" y1="49.53" x2="81.28" y2="49.53" width="0.4064" layer="16"/>
 <wire x1="85.09" y1="49.53" x2="82.55" y2="49.53" width="0.4064" layer="16"/>
@@
 <wire x1="78.74" y1="54.61" x2="78.74" y2="52.07" width="0.4064" layer="16"/>
 <wire x1="81.28" y1="49.53" x2="78.74" y2="52.07" width="0.4064" layer="16"/>
+<contactref element="E$59" pad="1"/>
+<contactref element="E$58" pad="1"/>
+<wire x1="85.09" y1="92.71" x2="82.55" y2="92.71" width="0.4064" layer="16"/>
+<contactref element="E$50" pad="2"/>
+<contactref element="E$4" pad="C"/>
+<wire x1="73.66" y1="97.79" x2="74.93" y2="96.52" width="0.4064" layer="16"/>
+<wire x1="63.5" y1="92.71" x2="62.23" y2="92.71" width="0.4064" layer="16"/>
+<wire x1="62.23" y1="92.71" x2="60.96" y2="93.98" width="0.4064" layer="16"/>
+<wire x1="69.85" y1="97.79" x2="73.66" y2="97.79" width="0.4064" layer="16"/>
+<wire x1="69.85" y1="95.25" x2="69.85" y2="97.79" width="0.4064" layer="16"/>
+<contactref element="E$44" pad="C"/>
+<wire x1="60.96" y1="97.79" x2="69.85" y2="97.79" width="0.4064" layer="16"/>
+<wire x1="60.96" y1="93.98" x2="60.96" y2="97.79" width="0.4064" layer="16"/>
+<contactref element="E$45" pad="C"/>
+<wire x1="58.42" y1="97.79" x2="60.96" y2="97.79" width="0.4064" layer="16"/>
+<wire x1="58.42" y1="96.52" x2="58.42" y2="97.79" width="0.4064" layer="16"/>
+<wire x1="49.53" y1="92.71" x2="50.8" y2="92.71" width="0.4064" layer="16"/>
+<wire x1="50.8" y1="92.71" x2="52.07" y2="93.98" width="0.4064" layer="16"/>
+<wire x1="54.61" y1="97.79" x2="58.42" y2="97.79" width="0.4064" layer="16"/>
+<wire x1="54.61" y1="96.52" x2="54.61" y2="97.79" width="0.4064" layer="16"/>
+<contactref element="E$1" pad="C"/>
+<wire x1="52.07" y1="97.79" x2="54.61" y2="97.79" width="0.4064" layer="16"/>
+<wire x1="52.07" y1="93.98" x2="52.07" y2="97.79" width="0.4064" layer="16"/>
 <contactref element="E$49" pad="2"/>
+<wire x1="43.18" y1="97.79" x2="52.07" y2="97.79" width="0.4064" layer="16"/>
+<wire x1="43.18" y1="95.25" x2="43.18" y2="97.79" width="0.4064" layer="16"/>
+<wire x1="39.37" y1="97.79" x2="43.18" y2="97.79" width="0.4064" layer="16"/>
 <wire x1="38.1" y1="96.52" x2="39.37" y2="97.79" width="0.4064" layer="16"/>
-<wire x1="85.09" y1="85.09" x2="78.74" y2="85.09" width="0.4064" layer="16"/>
-<wire x1="78.74" y1="85.09" x2="78.74" y2="86.36" width="0.4064" layer="16"/>
-</signal>
-<signal name="S$26">
-<contactref element="E$93" pad="2"/>
-<contactref element="E$58" pad="1"/>
-<wire x1="78.74" y1="96.52" x2="82.55" y2="92.71" width="0.4064" layer="16"/>
+<wire x1="82.55" y1="92.71" x2="78.74" y2="92.71" width="0.4064" layer="16"/>
+<wire x1="78.74" y1="92.71" x2="74.93" y2="96.52" width="0.4064" layer="16"/>
 </signal>
 </signals>
