File: microcap/pcb/testE.brd (EAGLE design)
At the start: 102 parts

Commit message: pcb test update
Parts:
- moved E$101 1.27 mm to (78.7, 91.4)
Connections:
- net S$8 renamed S$28
Routing:
- net S$28: track 199.4 -> 202.0 mm
- net S$18: track 305.4 -> 305.9 mm
Changed lines of the file:
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@@
 <element name="E$93" library="resistor" package="0207/10" value="" x="71.12" y="40.64" rot="R180.2"/>
 <element name="E$94" library="resistor" package="0207/10" value="" x="71.12" y="36.83" rot="R180.2"/>
-<element name="E$101" library="capacitor-wima" package="C5B2.5" value="" x="78.74" y="92.71" rot="R90"/>
+<element name="E$101" library="capacitor-wima" package="C5B2.5" value="" x="78.74" y="91.44" rot="R90"/>
 <element name="E$102" library="capacitor-wima" package="C2.5-2" value="" x="78.74" y="97.79"/>
 </elements>
@@
 <wire x1="76.2" y1="36.83" x2="76.2" y2="40.64" width="0.4064" layer="16"/>
 </signal>
-<signal name="S$8">
+<signal name="S$28">
+<contactref element="E$102" pad="1"/>
+<wire x1="76.2" y1="97.79" x2="77.47" y2="97.79" width="0.4064" layer="16"/>
+<contactref element="E$50" pad="2"/>
+<wire x1="74.93" y1="96.52" x2="76.2" y2="97.79" width="0.4064" layer="16"/>
+<contactref element="E$4" pad="C"/>
+<wire x1="73.66" y1="97.79" x2="74.93" y2="96.52" width="0.4064" layer="16"/>
+<wire x1="63.5" y1="92.71" x2="62.23" y2="92.71" width="0.4064" layer="16"/>
+<wire x1="62.23" y1="92.71" x2="60.96" y2="93.98" width="0.4064" layer="16"/>
+<wire x1="69.85" y1="97.79" x2="73.66" y2="97.79" width="0.4064" layer="16"/>
+<wire x1="69.85" y1="95.25" x2="69.85" y2="97.79" width="0.4064" layer="16"/>
+<contactref element="E$44" pad="C"/>
+<wire x1="60.96" y1="97.79" x2="69.85" y2="97.79" width="0.4064" layer="16"/>
+<wire x1="60.96" y1="93.98" x2="60.96" y2="97.79" width="0.4064" layer="16"/>
+<contactref element="E$45" pad="C"/>
+<wire x1="58.42" y1="97.79" x2="60.96" y2="97.79" width="0.4064" layer="16"/>
+<wire x1="58.42" y1="96.52" x2="58.42" y2="97.79" width="0.4064" layer="16"/>
+<wire x1="49.53" y1="92.71" x2="50.8" y2="92.71" width="0.4064" layer="16"/>
+<wire x1="50.8" y1="92.71" x2="52.07" y2="93.98" width="0.4064" layer="16"/>
+<wire x1="54.61" y1="97.79" x2="58.42" y2="97.79" width="0.4064" layer="16"/>
+<wire x1="54.61" y1="96.52" x2="54.61" y2="97.79" width="0.4064" layer="16"/>
+<contactref element="E$1" pad="C"/>
+<wire x1="52.07" y1="97.79" x2="54.61" y2="97.79" width="0.4064" layer="16"/>
+<wire x1="52.07" y1="93.98" x2="52.07" y2="97.79" width="0.4064" layer="16"/>
+<contactref element="E$49" pad="2"/>
+<wire x1="43.18" y1="97.79" x2="52.07" y2="97.79" width="0.4064" layer="16"/>
+<wire x1="43.18" y1="95.25" x2="43.18" y2="97.79" width="0.4064" layer="16"/>
+<wire x1="39.37" y1="97.79" x2="43.18" y2="97.79" width="0.4064" layer="16"/>
+<wire x1="38.1" y1="96.52" x2="39.37" y2="97.79" width="0.4064" layer="16"/>
+<wire x1="74.93" y1="96.52" x2="76.2" y2="95.25" width="0.4064" layer="16"/>
+<wire x1="76.2" y1="95.25" x2="76.2" y2="92.71" width="0.4064" layer="16"/>
 <contactref element="E$70" pad="1"/>
 <wire x1="85.09" y1="92.71" x2="85.09" y2="49.53" width="0.4064" layer="16"/>
@@
 <contactref element="E$58" pad="1"/>
 <wire x1="85.09" y1="92.71" x2="82.55" y2="92.71" width="0.4064" layer="16"/>
-<contactref element="E$50" pad="2"/>
-<contactref element="E$4" pad="C"/>
-<wire x1="73.66" y1="97.79" x2="74.93" y2="96.52" width="0.4064" layer="16"/>
-<wire x1="63.5" y1="92.71" x2="62.23" y2="92.71" width="0.4064" layer="16"/>
-<wire x1="62.23" y1="92.71" x2="60.96" y2="93.98" width="0.4064" layer="16"/>
-<wire x1="69.85" y1="97.79" x2="73.66" y2="97.79" width="0.4064" layer="16"/>
-<wire x1="69.85" y1="95.25" x2="69.85" y2="97.79" width="0.4064" layer="16"/>
-<contactref element="E$44" pad="C"/>
-<wire x1="60.96" y1="97.79" x2="69.85" y2="97.79" width="0.4064" layer="16"/>
-<wire x1="60.96" y1="93.98" x2="60.96" y2="97.79" width="0.4064" layer="16"/>
-<contactref element="E$45" pad="C"/>
-<wire x1="58.42" y1="97.79" x2="60.96" y2="97.79" width="0.4064" layer="16"/>
-<wire x1="58.42" y1="96.52" x2="58.42" y2="97.79" width="0.4064" layer="16"/>
-<wire x1="49.53" y1="92.71" x2="50.8" y2="92.71" width="0.4064" layer="16"/>
-<wire x1="50.8" y1="92.71" x2="52.07" y2="93.98" width="0.4064" layer="16"/>
-<wire x1="54.61" y1="97.79" x2="58.42" y2="97.79" width="0.4064" layer="16"/>
-<wire x1="54.61" y1="96.52" x2="54.61" y2="97.79" width="0.4064" layer="16"/>
-<contactref element="E$1" pad="C"/>
-<wire x1="52.07" y1="97.79" x2="54.61" y2="97.79" width="0.4064" layer="16"/>
-<wire x1="52.07" y1="93.98" x2="52.07" y2="97.79" width="0.4064" layer="16"/>
-<contactref element="E$49" pad="2"/>
-<wire x1="43.18" y1="97.79" x2="52.07" y2="97.79" width="0.4064" layer="16"/>
-<wire x1="43.18" y1="95.25" x2="43.18" y2="97.79" width="0.4064" layer="16"/>
-<wire x1="39.37" y1="97.79" x2="43.18" y2="97.79" width="0.4064" layer="16"/>
-<wire x1="38.1" y1="96.52" x2="39.37" y2="97.79" width="0.4064" layer="16"/>
-<wire x1="82.55" y1="92.71" x2="78.74" y2="92.71" width="0.4064" layer="16"/>
-<wire x1="78.74" y1="92.71" x2="74.93" y2="96.52" width="0.4064" layer="16"/>
+<wire x1="82.55" y1="92.71" x2="81.28" y2="92.71" width="0.4064" layer="16"/>
+<wire x1="81.28" y1="92.71" x2="80.01" y2="91.44" width="0.4064" layer="16"/>
 <contactref element="E$101" pad="1"/>
-<wire x1="78.74" y1="92.71" x2="78.74" y2="90.17" width="0.4064" layer="16"/>
-<wire x1="74.93" y1="96.52" x2="76.2" y2="97.79" width="0.4064" layer="16"/>
-<contactref element="E$102" pad="1"/>
-<wire x1="76.2" y1="97.79" x2="77.47" y2="97.79" width="0.4064" layer="16"/>
+<wire x1="78.74" y1="91.44" x2="78.74" y2="88.9" width="0.4064" layer="16"/>
+<wire x1="80.01" y1="91.44" x2="78.74" y2="91.44" width="0.4064" layer="16"/>
+<wire x1="77.47" y1="91.44" x2="78.74" y2="91.44" width="0.4064" layer="16"/>
+<wire x1="77.47" y1="91.44" x2="76.2" y2="92.71" width="0.4064" layer="16"/>
 </signal>
 <signal name="S$18">
@@
 <wire x1="106.68" y1="95.25" x2="80.01" y2="95.25" width="0.4064" layer="16"/>
 <contactref element="E$101" pad="2"/>
-<wire x1="80.01" y1="95.25" x2="78.74" y2="95.25" width="0.4064" layer="16"/>
+<wire x1="80.01" y1="95.25" x2="78.74" y2="93.98" width="0.4064" layer="16"/>
 <contactref element="E$102" pad="2"/>
 <wire x1="80.01" y1="97.79" x2="80.01" y2="95.25" width="0.4064" layer="16"/>

Commit message: pcb test update
Parts:
- moved E$101 1.27 mm to (78.7, 90.2)
Connections:
- net S$18 renamed S$8
Routing:
- net S$28: track 202.0 -> 203.8 mm
- net S$8: track 305.9 -> 307.2 mm
Changed lines of the file:
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@@
 <layer number="21" name="tPlace" color="7" fill="1" visible="yes" active="yes"/>
 <layer number="22" name="bPlace" color="7" fill="1" visible="yes" active="yes"/>
-<layer number="23" name="tOrigins" color="15" fill="1" visible="yes" active="yes"/>
-<layer number="24" name="bOrigins" color="15" fill="1" visible="yes" active="yes"/>
+<layer number="23" name="tOrigins" color="15" fill="1" visible="no" active="yes"/>
+<layer number="24" name="bOrigins" color="15" fill="1" visible="no" active="yes"/>
 <layer number="25" name="tNames" color="7" fill="1" visible="no" active="yes"/>
 <layer number="26" name="bNames" color="7" fill="1" visible="no" active="yes"/>
@@
 <element name="E$93" library="resistor" package="0207/10" value="" x="71.12" y="40.64" rot="R180.2"/>
 <element name="E$94" library="resistor" package="0207/10" value="" x="71.12" y="36.83" rot="R180.2"/>
-<element name="E$101" library="capacitor-wima" package="C5B2.5" value="" x="78.74" y="91.44" rot="R90"/>
+<element name="E$101" library="capacitor-wima" package="C5B2.5" value="" x="78.74" y="90.17" rot="R90"/>
 <element name="E$102" library="capacitor-wima" package="C2.5-2" value="" x="78.74" y="97.79"/>
 </elements>
@@
 <signal name="S$24">
 <polygon width="0.4064" layer="16">
-<vertex x="83.82" y="31.75"/>
+<vertex x="113.03" y="31.75"/>
 <vertex x="27.94" y="31.75"/>
-<vertex x="27.94" y="100.33"/>
-<vertex x="113.03" y="100.33"/>
-<vertex x="113.03" y="31.75"/>
+<vertex x="27.94" y="101.6"/>
+<vertex x="113.03" y="101.6"/>
 </polygon>
 </signal>
@@
 </signal>
 <signal name="S$28">
-<contactref element="E$102" pad="1"/>
-<wire x1="76.2" y1="97.79" x2="77.47" y2="97.79" width="0.4064" layer="16"/>
-<contactref element="E$50" pad="2"/>
-<wire x1="74.93" y1="96.52" x2="76.2" y2="97.79" width="0.4064" layer="16"/>
-<contactref element="E$4" pad="C"/>
-<wire x1="73.66" y1="97.79" x2="74.93" y2="96.52" width="0.4064" layer="16"/>
-<wire x1="63.5" y1="92.71" x2="62.23" y2="92.71" width="0.4064" layer="16"/>
-<wire x1="62.23" y1="92.71" x2="60.96" y2="93.98" width="0.4064" layer="16"/>
-<wire x1="69.85" y1="97.79" x2="73.66" y2="97.79" width="0.4064" layer="16"/>
-<wire x1="69.85" y1="95.25" x2="69.85" y2="97.79" width="0.4064" layer="16"/>
-<contactref element="E$44" pad="C"/>
-<wire x1="60.96" y1="97.79" x2="69.85" y2="97.79" width="0.4064" layer="16"/>
-<wire x1="60.96" y1="93.98" x2="60.96" y2="97.79" width="0.4064" layer="16"/>
-<contactref element="E$45" pad="C"/>
-<wire x1="58.42" y1="97.79" x2="60.96" y2="97.79" width="0.4064" layer="16"/>
-<wire x1="58.42" y1="96.52" x2="58.42" y2="97.79" width="0.4064" layer="16"/>
-<wire x1="49.53" y1="92.71" x2="50.8" y2="92.71" width="0.4064" layer="16"/>
-<wire x1="50.8" y1="92.71" x2="52.07" y2="93.98" width="0.4064" layer="16"/>
-<wire x1="54.61" y1="97.79" x2="58.42" y2="97.79" width="0.4064" layer="16"/>
-<wire x1="54.61" y1="96.52" x2="54.61" y2="97.79" width="0.4064" layer="16"/>
-<contactref element="E$1" pad="C"/>
-<wire x1="52.07" y1="97.79" x2="54.61" y2="97.79" width="0.4064" layer="16"/>
-<wire x1="52.07" y1="93.98" x2="52.07" y2="97.79" width="0.4064" layer="16"/>
-<contactref element="E$49" pad="2"/>
-<wire x1="43.18" y1="97.79" x2="52.07" y2="97.79" width="0.4064" layer="16"/>
-<wire x1="43.18" y1="95.25" x2="43.18" y2="97.79" width="0.4064" layer="16"/>
-<wire x1="39.37" y1="97.79" x2="43.18" y2="97.79" width="0.4064" layer="16"/>
-<wire x1="38.1" y1="96.52" x2="39.37" y2="97.79" width="0.4064" layer="16"/>
-<wire x1="74.93" y1="96.52" x2="76.2" y2="95.25" width="0.4064" layer="16"/>
-<wire x1="76.2" y1="95.25" x2="76.2" y2="92.71" width="0.4064" layer="16"/>
 <contactref element="E$70" pad="1"/>
 <wire x1="85.09" y1="92.71" x2="85.09" y2="49.53" width="0.4064" layer="16"/>
@@
 <wire x1="85.09" y1="92.71" x2="82.55" y2="92.71" width="0.4064" layer="16"/>
 <wire x1="82.55" y1="92.71" x2="81.28" y2="92.71" width="0.4064" layer="16"/>
-<wire x1="81.28" y1="92.71" x2="80.01" y2="91.44" width="0.4064" layer="16"/>
+<wire x1="81.28" y1="92.71" x2="78.74" y2="90.17" width="0.4064" layer="16"/>
 <contactref element="E$101" pad="1"/>
-<wire x1="78.74" y1="91.44" x2="78.74" y2="88.9" width="0.4064" layer="16"/>
-<wire x1="80.01" y1="91.44" x2="78.74" y2="91.44" width="0.4064" layer="16"/>
-<wire x1="77.47" y1="91.44" x2="78.74" y2="91.44" width="0.4064" layer="16"/>
-<wire x1="77.47" y1="91.44" x2="76.2" y2="92.71" width="0.4064" layer="16"/>
-</signal>
-<signal name="S$18">
+<wire x1="78.74" y1="90.17" x2="78.74" y2="87.63" width="0.4064" layer="16"/>
+<wire x1="78.74" y1="90.17" x2="77.47" y2="90.17" width="0.4064" layer="16"/>
+<wire x1="77.47" y1="90.17" x2="76.2" y2="91.44" width="0.4064" layer="16"/>
+<contactref element="E$102" pad="1"/>
+<wire x1="76.2" y1="95.25" x2="76.2" y2="91.44" width="0.4064" layer="16"/>
+<wire x1="76.2" y1="97.79" x2="77.47" y2="97.79" width="0.4064" layer="16"/>
+<contactref element="E$50" pad="2"/>
+<wire x1="74.93" y1="96.52" x2="76.2" y2="97.79" width="0.4064" layer="16"/>
+<wire x1="74.93" y1="96.52" x2="76.2" y2="95.25" width="0.4064" layer="16"/>
+<contactref element="E$4" pad="C"/>
+<wire x1="73.66" y1="97.79" x2="74.93" y2="96.52" width="0.4064" layer="16"/>
+<wire x1="63.5" y1="92.71" x2="62.23" y2="92.71" width="0.4064" layer="16"/>
+<wire x1="62.23" y1="92.71" x2="60.96" y2="93.98" width="0.4064" layer="16"/>
+<wire x1="69.85" y1="97.79" x2="73.66" y2="97.79" width="0.4064" layer="16"/>
+<wire x1="69.85" y1="95.25" x2="69.85" y2="97.79" width="0.4064" layer="16"/>
+<contactref element="E$44" pad="C"/>
+<wire x1="60.96" y1="97.79" x2="69.85" y2="97.79" width="0.4064" layer="16"/>
+<wire x1="60.96" y1="93.98" x2="60.96" y2="97.79" width="0.4064" layer="16"/>
+<contactref element="E$45" pad="C"/>
+<wire x1="58.42" y1="97.79" x2="60.96" y2="97.79" width="0.4064" layer="16"/>
+<wire x1="58.42" y1="96.52" x2="58.42" y2="97.79" width="0.4064" layer="16"/>
+<wire x1="49.53" y1="92.71" x2="50.8" y2="92.71" width="0.4064" layer="16"/>
+<wire x1="50.8" y1="92.71" x2="52.07" y2="93.98" width="0.4064" layer="16"/>
+<wire x1="54.61" y1="97.79" x2="58.42" y2="97.79" width="0.4064" layer="16"/>
+<wire x1="54.61" y1="96.52" x2="54.61" y2="97.79" width="0.4064" layer="16"/>
+<contactref element="E$1" pad="C"/>
+<wire x1="52.07" y1="97.79" x2="54.61" y2="97.79" width="0.4064" layer="16"/>
+<wire x1="52.07" y1="93.98" x2="52.07" y2="97.79" width="0.4064" layer="16"/>
+<contactref element="E$49" pad="2"/>
+<wire x1="43.18" y1="97.79" x2="52.07" y2="97.79" width="0.4064" layer="16"/>
+<wire x1="43.18" y1="95.25" x2="43.18" y2="97.79" width="0.4064" layer="16"/>
+<wire x1="39.37" y1="97.79" x2="43.18" y2="97.79" width="0.4064" layer="16"/>
+<wire x1="38.1" y1="96.52" x2="39.37" y2="97.79" width="0.4064" layer="16"/>
+</signal>
+<signal name="S$8">
+<contactref element="E$101" pad="2"/>
+<wire x1="78.74" y1="92.71" x2="78.74" y2="93.98" width="0.4064" layer="16"/>
 <wire x1="66.04" y1="36.83" x2="64.77" y2="36.83" width="0.4064" layer="16"/>
 <wire x1="69.85" y1="81.28" x2="68.58" y2="81.28" width="0.4064" layer="16"/>
@@
 <wire x1="107.95" y1="93.98" x2="106.68" y2="95.25" width="0.4064" layer="16"/>
 <wire x1="106.68" y1="95.25" x2="80.01" y2="95.25" width="0.4064" layer="16"/>
-<contactref element="E$101" pad="2"/>
-<wire x1="80.01" y1="95.25" x2="78.74" y2="93.98" width="0.4064" layer="16"/>
 <contactref element="E$102" pad="2"/>
 <wire x1="80.01" y1="97.79" x2="80.01" y2="95.25" width="0.4064" layer="16"/>
+<wire x1="78.74" y1="93.98" x2="80.01" y2="95.25" width="0.4064" layer="16"/>
 </signal>
 </signals>
