File: microcap/pcb/testF.brd (EAGLE design)
At the start: 103 parts

Commit message: pcb test update
Parts:
- moved E$102 45.8 mm to (33.0, 96.5)
Connections:
- removed net S$8: E$101.1, E$18.A, E$19.A, E$2.E, E$3.E, E$46.A, E$47.A, E$6.E, E$7.E, E$71.1, E$97.1
- new net S$30: E$101.1, E$102.1, E$18.A, E$19.A, E$2.E, E$3.E, E$46.A, E$47.A, E$6.E, E$7.E, E$71.1, E$97.1
- net S$29: now also E$102.2
Routing:
- net S$8: track 301.6 -> 0.00 mm
- net S$30: track 0.00 -> 288.9 mm
- net S$29: track 120.1 -> 125.9 mm
