File: microcap/pcb/testG.brd (EAGLE design)
At the start: 103 parts

Commit message: pcb test update
Parts:
- moved E$44 2.54 mm to (58.4, 94.0)
- moved E$45 2.54 mm to (54.6, 94.0)
- moved E$18 2.54 mm to (54.6, 43.2)
- moved E$19 2.54 mm to (58.4, 43.2)
- moved E$93 2.54 mm to (71.1, 38.1)
- moved E$1 1.27 mm to (43.2, 94.0)
- moved E$102 1.27 mm to (33.0, 97.8)
- moved E$4 1.27 mm to (69.8, 94.0)
- moved E$40 1.27 mm to (67.3, 94.0)
- moved E$42 1.27 mm to (52.1, 94.0)
- moved E$105 1.27 mm to (87.6, 55.9)
- moved E$20 1.27 mm to (34.3, 52.1)
- moved E$21 1.27 mm to (38.1, 57.1)
- moved E$22 1.27 mm to (74.9, 57.1)
- moved E$23 1.27 mm to (78.7, 52.1)
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Connections:
- removed net S$29: E$1.C, E$101.2, E$102.2, E$29.1, E$4.C, E$44.C, E$45.C, E$49.2, E$50.2, E$58.1, E$59.1
- removed net S$30: E$101.1, E$102.1, E$18.A, E$19.A, E$2.E, E$3.E, E$46.A, E$47.A, E$6.E, E$7.E, E$71.1, E$97.1
- new net S$28: E$105.C, E$16.C, E$17.C, E$21.2, E$22.2, E$5.C, E$70.1, E$8.C
- new net S$8: E$45.A, E$46.C
- net S$18: now also E$1.C, E$101.2, E$102.2, E$29.1, E$4.C, E$44.C, E$45.C, E$49.2, E$50.2, E$58.1, E$59.1; no longer E$16.C, E$17.C, E$21.2, E$22.2, E$5.C, E$70.1, E$8.C
- net S$22: now also E$44.A, E$47.C; no longer E$45.A, E$46.C
- net S$25: now also E$101.1, E$102.1, E$18.A, E$19.A, E$2.E, E$3.E, E$46.A, E$47.A, E$6.E, E$7.E, E$71.1, E$97.1; no longer E$44.A, E$47.C
Routing:
- net S$25: track 2.54 -> 296.8 mm
- net S$30: track 288.9 -> 0.00 mm
- net S$29: track 125.9 -> 0.00 mm
- net S$28: track 0.00 -> 90.6 mm
- net S$18: track 82.2 -> 133.8 mm
- net S$8: track 0.00 -> 5.08 mm, vias 0 -> 2
- net S$12: track 2.54 -> 6.35 mm, vias 0 -> 2
- net S$22: track 2.54 -> 5.08 mm, vias 0 -> 2
- net S$19: track 2.54 -> 5.08 mm, vias 0 -> 2
- net S$26: track 35.9 -> 37.7 mm
- net S$36: track 59.6 -> 60.8 mm
- net S$23: track 51.9 -> 53.2 mm
- net S$20: track 8.67 -> 9.94 mm
- net S$15: track 4.34 -> 3.81 mm
- net S$27: vias 1 -> 0
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