File: microcap/pcb/tmp.brd (EAGLE design)
At the start: 408 parts

Commit message: pcb test update
Parts:
- removed E$1, E$103, E$104, E$105, E$106, E$120, E$121, E$122, E$123, E$137, E$138, E$139, E$140, E$154, E$155, E$156, E$157, E$171, E$172, E$173, E$174, E$188, E$189, E$190, E$191, E$2, E$205, E$206, E$22, E$23, E$24, E$25, E$3, E$39, E$4, E$5, E$52, E$53, E$54, E$6, E$68, E$69, E$7, E$70, E$71, E$8, E$85, E$86, E$87, E$88: (no value), transistor:TO92-CBE
- removed E$10, E$107, E$108, E$109, E$11, E$110, E$12, E$124, E$125, E$126, E$127, E$141, E$142, E$143, E$144, E$158, E$159, E$160, E$161, E$175, E$176, E$177, E$178, E$192, E$193, E$194, E$195, E$26, E$27, E$28, E$29, E$40, E$41, E$42, E$43, E$55, E$56, E$57, E$58, E$72, E$73, E$74, E$75, E$89, E$9, E$90, E$91, E$92: (no value), transistor:T-30_V
- removed E$100, E$101, E$102, E$115, E$116, E$117, E$118, E$119, E$132, E$133, E$134, E$135, E$136, E$149, E$150, E$151, E$152, E$153, E$166, E$167, E$168, E$169, E$17, E$170, E$18, E$183, E$184, E$185, E$186, E$187, E$19, E$20, E$200, E$201, E$202, E$203, E$204, E$21, E$34, E$35, E$36, E$37, E$38, E$48, E$49, E$50, E$51, E$63, E$64, E$65, E$66, E$67, E$80, E$81, E$82, E$83, E$84, E$93, E$98, E$99: (no value), resistor:0207/10
- removed E$111, E$112, E$113, E$114, E$128, E$129, E$13, E$130, E$131, E$14, E$145, E$146, E$147, E$148, E$15, E$16, E$162, E$163, E$164, E$165, E$179, E$180, E$181, E$182, E$196, E$197, E$198, E$199, E$30, E$31, E$32, E$33, E$44, E$45, E$46, E$47, E$59, E$60, E$61, E$62, E$76, E$77, E$78, E$79, E$94, E$95, E$96, E$97: (no value), diode:C2992
- added E$409, E$512, E$615, E$718, E$821: (no value), capacitor-wima:C5B2.5
- added E$410, E$425, E$426, E$427, E$428, E$441, E$442, E$443, E$444, E$511, E$513, E$528, E$529, E$530, E$531, E$544, E$545, E$546, E$547, E$614, E$616, E$631, E$632, E$633, E$634, E$647, E$648, E$649, E$650, E$717, E$719, E$734, E$735, E$736, E$737, E$750, E$751, E$752, E$753, E$820, E$822: (no value), resistor:0207/10
- added E$411, E$514, E$617, E$720, E$823: (no value), capacitor-wima:C2.5-2
- added E$412, E$515, E$618, E$721, E$824: (no value), diode:ZDIO-10
- added E$413, E$414, E$415, E$416, E$429, E$430, E$431, E$432, E$516, E$517, E$518, E$519, E$532, E$533, E$534, E$535, E$619, E$620, E$621, E$622, E$635, E$636, E$637, E$638, E$722, E$723, E$724, E$725, E$738, E$739, E$740, E$741: (no value), transistor:TO92-CBE
- added E$417, E$418, E$419, E$420, E$433, E$434, E$435, E$436, E$520, E$521, E$522, E$523, E$536, E$537, E$538, E$539, E$623, E$624, E$625, E$626, E$639, E$640, E$641, E$642, E$726, E$727, E$728, E$729, E$742, E$743, E$744, E$745: (no value), transistor:T-30_V
- added E$421, E$422, E$423, E$424, E$437, E$438, E$439, E$440, E$524, E$525, E$526, E$527, E$540, E$541, E$542, E$543, E$627, E$628, E$629, E$630, E$643, E$644, E$645, E$646, E$730, E$731, E$732, E$733, E$746, E$747, E$748, E$749: (no value), diode:C2992
- added E$445, E$446, E$447, E$448, E$449, E$450, E$451, E$452, E$453, E$454, E$455, E$456, E$457, E$458, E$459, E$460, E$461, E$462, E$463, E$464, E$465, E$466, E$467, E$468, E$469, E$470, E$471, E$472, E$473, E$474, E$475, E$476, E$477, E$478, E$479, E$480, E$481, E$482, E$483, E$484, E$485, E$486, E$487, E$488, E$489, E$490, E$491, E$492, E$493, E$494, E$495, E$496, E$497, E$498, E$499, E$500, E$501, E$502, E$503, E$504, E$505, E$506, E$507, E$508, E$509, E$510, E$548, E$549, E$550, E$551, E$552, E$553, E$554, E$555, E$556, E$557, E$558, E$559, E$560, E$561, E$562, E$563, E$564, E$565, E$566, E$567, E$568, E$569, E$570, E$571, E$572, E$573, E$574, E$575, E$576, E$577, E$578, E$579, E$580, E$581, E$582, E$583, E$584, E$585, E$586, E$587, E$588, E$589, E$590, E$591, E$592, E$593, E$594, E$595, E$596, E$597, E$598, E$599, E$600, E$601, E$602, E$603, E$604, E$605, E$606, E$607, E$608, E$609, E$610, E$611, E$612, E$613, E$651, E$652, E$653, E$654, E$655, E$656, E$657, E$658, E$659, E$660, E$661, E$662, E$663, E$664, E$665, E$666, E$667, E$668, E$669, E$670, E$671, E$672, E$673, E$674, E$675, E$676, E$677, E$678, E$679, E$680, E$681, E$682, E$683, E$684, E$685, E$686, E$687, E$688, E$689, E$690, E$691, E$692, E$693, E$694, E$695, E$696, E$697, E$698, E$699, E$700, E$701, E$702, E$703, E$704, E$705, E$706, E$707, E$708, E$709, E$710, E$711, E$712, E$713, E$714, E$715, E$716, E$754, E$755, E$756, E$757, E$758, E$759, E$760, E$761, E$762, E$763, E$764, E$765, E$766, E$767, E$768, E$769, E$770, E$771, E$772, E$773, E$774, E$775, E$776, E$777, E$778, E$779, E$780, E$781, E$782, E$783, E$784, E$785, E$786, E$787, E$788, E$789, E$790, E$791, E$792, E$793, E$794, E$795, E$796, E$797, E$798, E$799, E$800, E$801, E$802, E$803, E$804, E$805, E$806, E$807, E$808, E$809, E$810, E$811, E$812, E$813, E$814, E$815, E$816, E$817, E$818, E$819: (no value), pinhead:1X01
- E$209, E$210, E$226, E$311, E$312, E$313, E$328, E$329: device transistor:T-30_V -> transistor:TO92-CBE
- E$213, E$214, E$230, E$315, E$316, E$317, E$332, E$333: device diode:C2992 -> transistor:T-30_V
- E$217, E$218, E$234, E$319, E$320, E$321, E$336, E$337: device resistor:0207/10 -> diode:C2992
- E$222, E$307, E$324, E$325, E$341: device transistor:TO92-CBE -> resistor:0207/10
- E$239, E$240, E$241, E$242, E$256, E$257, E$258, E$259, E$273, E$274, E$275, E$276, E$290, E$291, E$292, E$293, E$342, E$343, E$344, E$358, E$359, E$360, E$361, E$375, E$376, E$377, E$378, E$392, E$393, E$394, E$395: device transistor:TO92-CBE -> pinhead:1X01
- E$243, E$244, E$245, E$246, E$260, E$261, E$262, E$263, E$277, E$278, E$279, E$280, E$294, E$295, E$296, E$297, E$345, E$346, E$347, E$348, E$362, E$363, E$364, E$365, E$379, E$380, E$381, E$382, E$396, E$397, E$398, E$399: device transistor:T-30_V -> pinhead:1X01
- E$247, E$248, E$249, E$250, E$264, E$265, E$266, E$267, E$281, E$282, E$283, E$284, E$298, E$299, E$300, E$301, E$349, E$350, E$351, E$352, E$366, E$367, E$368, E$369, E$383, E$384, E$385, E$386, E$400, E$401, E$402, E$403: device diode:C2992 -> pinhead:1X01
- E$251, E$252, E$253, E$254, E$255, E$268, E$269, E$270, E$271, E$272, E$285, E$286, E$287, E$288, E$289, E$302, E$303, E$304, E$353, E$354, E$355, E$356, E$357, E$370, E$371, E$372, E$373, E$374, E$387, E$388, E$389, E$390, E$391, E$404, E$405, E$406, E$407: device resistor:0207/10 -> pinhead:1X01
- E$306: device resistor:0207/10 -> capacitor-wima:C5B2.5
- E$308: device transistor:TO92-CBE -> capacitor-wima:C2.5-2
- E$309: device transistor:TO92-CBE -> diode:ZDIO-10
- moved E$404 336.8 mm to (201.9, 12.7), turned to 0 degrees
- moved E$405 324.9 mm to (201.9, 10.2), turned to 0 degrees
- moved E$402 320.7 mm to (201.9, 17.8), turned to 0 degrees
- moved E$394 319.3 mm to (201.9, -12.7), turned to 0 degrees
- moved E$403 316.1 mm to (201.9, 15.2), turned to 0 degrees
- moved E$392 312.0 mm to (201.9, -7.62), turned to 0 degrees
- moved E$398 308.4 mm to (201.9, 2.54), turned to 0 degrees
- moved E$397 306.8 mm to (201.9, -20.3), turned to 0 degrees
- moved E$387 304.6 mm to (201.9, -35.6), turned to 0 degrees
- moved E$401 303.3 mm to (201.9, -5.08), turned to 0 degrees
- moved E$400 301.0 mm to (201.9, -2.54), turned to 0 degrees
- moved E$399 296.0 mm to (201.9, 0.00), turned to 0 degrees
- moved E$406 291.4 mm to (201.9, 7.62), turned to 0 degrees
- moved E$393 287.7 mm to (201.9, -10.2), turned to 0 degrees
- moved E$407 286.8 mm to (201.9, 5.08), turned to 0 degrees
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Connections:
- removed net S$1: E$48.1
- removed net S$10: E$1.E
- removed net S$109: E$140.E
- removed net S$11: E$18.1, E$5.B, E$7.C
- removed net S$117: E$149.1
- removed net S$12: E$5.E
- removed net S$125: E$155.B, E$169.2
- removed net S$126: E$163.A, E$164.C
- removed net S$138: E$172.B, E$186.2
- removed net S$14: E$8.E
- removed net S$146: E$188.B, E$190.C, E$201.1
- removed net S$147: E$188.E
- removed net S$15: E$19.1, E$6.C, E$8.B
- removed net S$154: E$188.C, E$191.C, E$196.C, E$197.C, E$201.2, E$202.2, E$204.2
- removed net S$155: E$189.E, E$190.E, E$198.A, E$199.A
- removed net S$16: E$17.2, E$7.B
- removed net S$167: E$205.C, E$208.C, E$213.C, E$214.C, E$218.2, E$219.2, E$221.2
- removed net S$17: E$20.2, E$6.B
- removed net S$175: E$223.C, E$225.B, E$236.1
- removed net S$176: E$224.B, E$234.2
- removed net S$18: E$1.C, E$4.C, E$44.C, E$45.C, E$49.2, E$50.2, E$93.2
- removed net S$19: E$14.A, E$15.C
- removed net S$2: E$2.C, E$4.B, E$50.1
- removed net S$20: E$13.A, E$16.C
- removed net S$204: E$265.A, E$266.C
- removed net S$205: E$264.A, E$267.C
- removed net S$21: E$13.C, E$14.C, E$18.2, E$19.2, E$21.2, E$5.C, E$8.C
- removed net S$212: E$273.E
- removed net S$213: E$276.E
- removed net S$22: E$45.A, E$46.C
- removed net S$225: E$290.E
- removed net S$23: E$15.A, E$16.A, E$6.E, E$7.E
- removed net S$233: E$291.E, E$292.E, E$300.A, E$301.A
- removed net S$234: E$302.1
- removed net S$237: E$307.B, E$309.C, E$320.1
- removed net S$238: E$307.E
- removed net S$239: E$310.E
- removed net S$24: E$17.1
- removed net S$240: E$308.C, E$310.B, E$321.1
- removed net S$241: E$309.B, E$319.2
- removed net S$242: E$308.B, E$322.2
- removed net S$243: E$316.A, E$317.C
- removed net S$244: E$315.A, E$318.C
- removed net S$245: E$307.C, E$310.C, E$315.C, E$316.C, E$320.2, E$321.2, E$323.2
- removed net S$246: E$308.E, E$309.E, E$317.A, E$318.A
- removed net S$247: E$319.1
- removed net S$25: E$44.A, E$47.C
- removed net S$250: E$324.B, E$326.C, E$337.1
- removed net S$251: E$324.E
- removed net S$252: E$327.E
- removed net S$253: E$325.C, E$327.B, E$338.1
- removed net S$254: E$326.B, E$336.2
- removed net S$255: E$325.B, E$339.2
- removed net S$256: E$333.A, E$334.C
- removed net S$257: E$332.A, E$335.C
- removed net S$258: E$324.C, E$327.C, E$332.C, E$333.C, E$337.2, E$338.2, E$340.2
- removed net S$259: E$325.E, E$326.E, E$334.A, E$335.A
- removed net S$260: E$336.1
- removed net S$263: E$341.B, E$343.C, E$354.1
- removed net S$264: E$341.E
- removed net S$265: E$344.E
- removed net S$266: E$342.C, E$344.B, E$355.1
- removed net S$267: E$343.B, E$353.2
- removed net S$268: E$342.B, E$356.2
- removed net S$269: E$350.A, E$351.C
- removed net S$270: E$349.A, E$352.C
- removed net S$271: E$341.C, E$344.C, E$349.C, E$350.C, E$354.2, E$355.2, E$357.2
- removed net S$272: E$342.E, E$343.E, E$351.A, E$352.A
- removed net S$273: E$353.1
- removed net S$276: E$358.B, E$360.C, E$371.1
- removed net S$277: E$358.E
- removed net S$278: E$361.E
- removed net S$279: E$359.C, E$361.B, E$372.1
- removed net S$280: E$360.B, E$370.2
- removed net S$281: E$359.B, E$373.2
- removed net S$282: E$367.A, E$368.C
- removed net S$283: E$366.A, E$369.C
- removed net S$284: E$358.C, E$361.C, E$366.C, E$367.C, E$371.2, E$372.2, E$374.2
- removed net S$285: E$359.E, E$360.E, E$368.A, E$369.A
- removed net S$286: E$370.1
- removed net S$289: E$375.B, E$377.C, E$388.1
- removed net S$29: E$22.B, E$24.C, E$35.1
- removed net S$290: E$375.E
- removed net S$291: E$378.E
- removed net S$292: E$376.C, E$378.B, E$389.1
- removed net S$293: E$377.B, E$387.2
- removed net S$294: E$376.B, E$390.2
- removed net S$295: E$384.A, E$385.C
- removed net S$296: E$383.A, E$386.C
- removed net S$297: E$375.C, E$378.C, E$383.C, E$384.C, E$388.2, E$389.2, E$391.2
- removed net S$298: E$376.E, E$377.E, E$385.A, E$386.A
- removed net S$299: E$387.1
- removed net S$3: E$2.E, E$3.E, E$46.A, E$47.A
- removed net S$30: E$22.E
- removed net S$302: E$392.B, E$394.C, E$405.1
- removed net S$303: E$392.E
- removed net S$304: E$395.E
- removed net S$305: E$393.C, E$395.B, E$406.1
- removed net S$306: E$394.B, E$404.2
- removed net S$307: E$393.B, E$407.2
- removed net S$308: E$401.A, E$402.C
- removed net S$309: E$400.A, E$403.C
- removed net S$31: E$25.E
- removed net S$310: E$392.C, E$395.C, E$400.C, E$401.C, E$405.2, E$406.2, E$408.2
- removed net S$311: E$393.E, E$394.E, E$402.A, E$403.A
- removed net S$312: E$404.1
- removed net S$32: E$23.C, E$25.B, E$36.1
- removed net S$33: E$24.B, E$34.2
- removed net S$34: E$23.B, E$37.2
- removed net S$35: E$31.A, E$32.C
- removed net S$36: E$30.A, E$33.C
- removed net S$37: E$22.C, E$25.C, E$30.C, E$31.C, E$35.2, E$36.2, E$38.2
- removed net S$38: E$23.E, E$24.E, E$32.A, E$33.A
- removed net S$39: E$34.1
- removed net S$4: E$4.E
- removed net S$42: E$39.B, E$53.C, E$64.1
- removed net S$43: E$39.E
- removed net S$44: E$54.E
- removed net S$45: E$52.C, E$54.B, E$65.1
- removed net S$46: E$53.B, E$63.2
- removed net S$47: E$52.B, E$66.2
- removed net S$48: E$60.A, E$61.C
- removed net S$49: E$59.A, E$62.C
- removed net S$5: E$3.B, E$48.2
- removed net S$50: E$39.C, E$54.C, E$59.C, E$60.C, E$64.2, E$65.2, E$67.2
- removed net S$51: E$52.E, E$53.E, E$61.A, E$62.A
- removed net S$52: E$63.1
- removed net S$55: E$68.B, E$70.C, E$81.1
- removed net S$56: E$68.E
- removed net S$57: E$71.E
- removed net S$58: E$69.C, E$71.B, E$82.1
- removed net S$59: E$70.B, E$80.2
- removed net S$6: E$2.B, E$51.2
- removed net S$60: E$69.B, E$83.2
- removed net S$68: E$85.B, E$87.C, E$99.1
- removed net S$88: E$111.A, E$114.C
- removed net S$89: E$103.C, E$106.C, E$111.C, E$112.C, E$116.2, E$117.2, E$119.2
- removed net S$9: E$1.B, E$3.C, E$49.1
- removed net S$96: E$123.E
- removed net S$97: E$121.C, E$123.B, E$134.1
- new net S$105: E$334.A, E$337.C
- new net S$106: E$338.1, E$373.1
- new net S$119: E$413.B, E$415.C, E$426.1
- new net S$131: E$430.B, E$444.2
- new net S$132: E$431.B, E$441.2
- new net S$144: E$429.C, E$432.C, E$437.C, E$438.C, E$442.2, E$443.2, E$480.1, E$515.C
- new net S$145: E$444.1, E$477.1
- new net S$157: E$532.E
- new net S$158: E$535.E
- new net S$170: E$517.E, E$518.E, E$526.A, E$527.A, E$533.E, E$534.E, E$542.A, E$543.A, E$584.1, E$610.1, E$615.1, E$617.1
- new net S$171: E$525.A, E$526.C
- new net S$197: E$694.1
- new net S$209: E$723.C, E$725.B, E$736.1
- new net S$210: E$724.B, E$734.2
- new net S$222: E$750.1, E$785.1
- new net S$223: E$737.1, E$783.1
- new net S$66: E$208.B, E$222.2
- new net S$79: E$219.1, E$269.1
- new net S$92: E$313.E
- new net S$93: E$311.C, E$313.B, E$324.1
- net S$100: now also E$329.E; no longer E$129.A, E$130.C
- net S$101: now also E$327.C, E$329.B, E$340.1; no longer E$128.A, E$131.C
- net S$102: now also E$327.B, E$341.2; no longer E$120.C, E$123.C, E$128.C, E$129.C, E$133.2, E$134.2, E$136.2
- net S$103: now also E$328.B, E$338.2; no longer E$121.E, E$122.E, E$130.A, E$131.A
- net S$104: now also E$335.A, E$336.C; no longer E$132.1
- net S$107: now also E$325.1, E$371.1; no longer E$137.B, E$139.C, E$150.1
- net S$108: now also E$322.1, E$372.1; no longer E$137.E
- net S$110: now also E$385.1; no longer E$138.C, E$140.B, E$151.1
- net S$111: now also E$310.C, E$313.C, E$318.C, E$319.C, E$323.2, E$324.2, E$347.1, E$362.1, E$363.1, E$409.2, E$411.2; no longer E$139.B, E$149.2
- net S$112: now also E$311.E, E$312.E, E$320.A, E$321.A, E$327.E, E$328.E, E$336.A, E$337.A, E$378.1, E$404.1, E$409.1, E$411.1; no longer E$138.B, E$152.2
- net S$113: now also E$319.A, E$320.C; no longer E$146.A, E$147.C
- net S$114: now also E$318.A, E$321.C; no longer E$145.A, E$148.C
- net S$115: now also E$326.C, E$329.C, E$334.C, E$335.C, E$339.2, E$340.2, E$377.1, E$412.C; no longer E$137.C, E$140.C, E$145.C, E$146.C, E$150.2, E$151.2, E$153.2
- net S$116: now also E$341.1, E$374.1; no longer E$138.E, E$139.E, E$147.A, E$148.A
- net S$120: now also E$413.E; no longer E$154.B, E$156.C, E$167.1
- net S$121: now also E$416.E; no longer E$154.E
- net S$122: now also E$414.C, E$416.B, E$427.1; no longer E$157.E
- net S$123: now also E$415.B, E$425.2; no longer E$155.C, E$157.B, E$168.1
- net S$124: now also E$414.B, E$428.2; no longer E$156.B, E$166.2
- net S$127: now also E$429.B, E$431.C, E$442.1; no longer E$162.A, E$165.C
- net S$128: now also E$429.E; no longer E$154.C, E$157.C, E$162.C, E$163.C, E$167.2, E$168.2, E$170.2
- net S$129: now also E$432.E; no longer E$155.E, E$156.E, E$164.A, E$165.A
- net S$130: now also E$430.C, E$432.B, E$443.1; no longer E$166.1
- net S$133: now also E$438.A, E$439.C; no longer E$171.B, E$173.C, E$184.1
- net S$134: now also E$437.A, E$440.C; no longer E$171.E
- net S$135: now also E$441.1, E$476.1; no longer E$174.E
- net S$136: now also E$428.1, E$474.1; no longer E$172.C, E$174.B, E$185.1
- net S$137: now also E$425.1, E$475.1; no longer E$173.B, E$183.2
- net S$139: now also E$488.1; no longer E$180.A, E$181.C
- net S$140: now also E$413.C, E$416.C, E$421.C, E$422.C, E$426.2, E$427.2, E$450.1, E$465.1, E$466.1, E$512.2, E$514.2; no longer E$179.A, E$182.C
- net S$141: now also E$414.E, E$415.E, E$423.A, E$424.A, E$430.E, E$431.E, E$439.A, E$440.A, E$481.1, E$507.1, E$512.1, E$514.1; no longer E$171.C, E$174.C, E$179.C, E$180.C, E$184.2, E$185.2, E$187.2
- net S$142: now also E$422.A, E$423.C; no longer E$172.E, E$173.E, E$181.A, E$182.A
- net S$143: now also E$421.A, E$424.C; no longer E$183.1
- net S$148: now also E$516.B, E$518.C, E$529.1; no longer E$191.E
- net S$149: now also E$516.E; no longer E$189.C, E$191.B, E$202.1
- net S$150: now also E$519.E; no longer E$190.B, E$200.2
- net S$151: now also E$517.C, E$519.B, E$530.1; no longer E$189.B, E$203.2
- net S$152: now also E$518.B, E$528.2; no longer E$197.A, E$198.C
- net S$153: now also E$517.B, E$531.2; no longer E$196.A, E$199.C
- net S$156: now also E$532.B, E$534.C, E$545.1; no longer E$200.1
- net S$159: now also E$533.C, E$535.B, E$546.1; no longer E$205.B, E$207.C, E$218.1
- net S$160: now also E$533.B, E$547.2; no longer E$205.E
- net S$161: now also E$534.B, E$544.2; no longer E$208.E
- net S$162: now also E$541.A, E$542.C; no longer E$206.C, E$208.B, E$219.1
- net S$163: now also E$540.A, E$543.C; no longer E$207.B, E$217.2
- net S$164: now also E$544.1, E$579.1; no longer E$206.B, E$220.2
- net S$165: now also E$531.1, E$577.1; no longer E$214.A, E$215.C
- net S$166: now also E$528.1, E$578.1; no longer E$213.A, E$216.C
- net S$168: now also E$591.1; no longer E$206.E, E$207.E, E$215.A, E$216.A
- net S$169: now also E$516.C, E$519.C, E$524.C, E$525.C, E$529.2, E$530.2, E$553.1, E$568.1, E$569.1, E$615.2, E$617.2; no longer E$217.1
- net S$172: now also E$524.A, E$527.C; no longer E$222.B, E$224.C, E$235.1
- net S$173: now also E$532.C, E$535.C, E$540.C, E$541.C, E$545.2, E$546.2, E$583.1, E$618.C; no longer E$222.E
- net S$174: now also E$547.1, E$580.1; no longer E$225.E
- net S$177: now also E$619.B, E$621.C, E$632.1; no longer E$223.B, E$237.2
- net S$178: now also E$619.E; no longer E$231.A, E$232.C
- net S$179: now also E$622.E; no longer E$230.A, E$233.C
- net S$180: now also E$620.C, E$622.B, E$633.1; no longer E$222.C, E$225.C, E$230.C, E$231.C, E$235.2, E$236.2, E$238.2
- net S$181: now also E$621.B, E$631.2; no longer E$223.E, E$224.E, E$232.A, E$233.A
- net S$182: now also E$620.B, E$634.2; no longer E$234.1
- net S$185: now also E$635.B, E$637.C, E$648.1; no longer E$239.B, E$241.C, E$252.1
- net S$186: now also E$635.E; no longer E$239.E
- net S$187: now also E$638.E; no longer E$242.E
- net S$188: now also E$636.C, E$638.B, E$649.1; no longer E$240.C, E$242.B, E$253.1
- net S$189: now also E$636.B, E$650.2; no longer E$241.B, E$251.2
- net S$190: now also E$637.B, E$647.2; no longer E$240.B, E$254.2
- net S$191: now also E$644.A, E$645.C; no longer E$248.A, E$249.C
- net S$192: now also E$643.A, E$646.C; no longer E$247.A, E$250.C
- net S$193: now also E$647.1, E$682.1; no longer E$239.C, E$242.C, E$247.C, E$248.C, E$252.2, E$253.2, E$255.2
- net S$194: now also E$634.1, E$680.1; no longer E$240.E, E$241.E, E$249.A, E$250.A
- net S$195: now also E$631.1, E$681.1; no longer E$251.1
- net S$198: now also E$619.C, E$622.C, E$627.C, E$628.C, E$632.2, E$633.2, E$656.1, E$671.1, E$672.1, E$718.2, E$720.2; no longer E$256.B, E$258.C, E$269.1
- net S$199: now also E$620.E, E$621.E, E$629.A, E$630.A, E$636.E, E$637.E, E$645.A, E$646.A, E$687.1, E$713.1, E$718.1, E$720.1; no longer E$256.E
- net S$200: now also E$628.A, E$629.C; no longer E$259.E
- net S$201: now also E$627.A, E$630.C; no longer E$257.C, E$259.B, E$270.1
- net S$202: now also E$635.C, E$638.C, E$643.C, E$644.C, E$648.2, E$649.2, E$686.1, E$721.C; no longer E$258.B, E$268.2
- net S$203: now also E$650.1, E$683.1; no longer E$257.B, E$271.2
- net S$206: now also E$722.B, E$724.C, E$735.1; no longer E$256.C, E$259.C, E$264.C, E$265.C, E$269.2, E$270.2, E$272.2
- net S$207: now also E$722.E; no longer E$257.E, E$258.E, E$266.A, E$267.A
- net S$208: now also E$725.E; no longer E$268.1
- net S$211: now also E$723.B, E$737.2; no longer E$273.B, E$275.C, E$286.1
- net S$214: now also E$738.B, E$740.C, E$751.1; no longer E$274.C, E$276.B, E$287.1
- net S$215: now also E$738.E; no longer E$275.B, E$285.2
- net S$216: now also E$741.E; no longer E$274.B, E$288.2
- net S$217: now also E$739.C, E$741.B, E$752.1; no longer E$282.A, E$283.C
- net S$218: now also E$739.B, E$753.2; no longer E$281.A, E$284.C
- net S$219: now also E$740.B, E$750.2; no longer E$273.C, E$276.C, E$281.C, E$282.C, E$286.2, E$287.2, E$289.2
- net S$220: now also E$747.A, E$748.C; no longer E$274.E, E$275.E, E$283.A, E$284.A
- net S$221: now also E$746.A, E$749.C; no longer E$285.1
- net S$224: now also E$734.1, E$784.1; no longer E$290.B, E$292.C, E$303.1
- net S$226: now also E$797.1; no longer E$293.E
- net S$227: now also E$722.C, E$725.C, E$730.C, E$731.C, E$735.2, E$736.2, E$759.1, E$774.1, E$775.1, E$821.2, E$823.2; no longer E$291.C, E$293.B, E$304.1
- net S$228: now also E$723.E, E$724.E, E$732.A, E$733.A, E$739.E, E$740.E, E$748.A, E$749.A, E$790.1, E$816.1, E$821.1, E$823.1; no longer E$292.B, E$302.2
- net S$229: now also E$731.A, E$732.C; no longer E$291.B, E$305.2
- net S$230: now also E$730.A, E$733.C; no longer E$299.A, E$300.C
- net S$231: now also E$738.C, E$741.C, E$746.C, E$747.C, E$751.2, E$752.2, E$789.1, E$824.C; no longer E$298.A, E$301.C
- net S$232: now also E$753.1, E$786.1; no longer E$290.C, E$293.C, E$298.C, E$299.C, E$303.2, E$304.2, E$306.2
- net S$61: now also E$207.B, E$209.C, E$220.1; no longer E$77.A, E$78.C
- net S$62: now also E$207.E; no longer E$76.A, E$79.C
- net S$63: now also E$210.E; no longer E$68.C, E$71.C, E$76.C, E$77.C, E$81.2, E$82.2, E$84.2
- net S$64: now also E$208.C, E$210.B, E$221.1; no longer E$69.E, E$70.E, E$78.A, E$79.A
- net S$65: now also E$209.B, E$219.2; no longer E$80.1
- net S$69: now also E$223.B, E$225.C, E$236.1; no longer E$85.E
- net S$70: now also E$223.E; no longer E$88.E
- net S$71: now also E$226.E; no longer E$100.1, E$86.C, E$88.B
- net S$72: now also E$224.C, E$226.B, E$237.1; no longer E$87.B, E$98.2
- net S$73: now also E$224.B, E$238.2; no longer E$101.2, E$86.B
- net S$74: now also E$225.B, E$235.2; no longer E$95.A, E$96.C
- net S$75: now also E$232.A, E$233.C; no longer E$94.A, E$97.C
- net S$76: now also E$231.A, E$234.C; no longer E$100.2, E$102.2, E$85.C, E$88.C, E$94.C, E$95.C, E$99.2
- net S$77: now also E$235.1, E$270.1; no longer E$86.E, E$87.E, E$96.A, E$97.A
- net S$78: now also E$222.1, E$268.1; no longer E$98.1
- net S$81: now also E$282.1; no longer E$103.B, E$105.C, E$116.1
- net S$82: now also E$207.C, E$210.C, E$215.C, E$216.C, E$220.2, E$221.2, E$244.1, E$259.1, E$260.1, E$306.2, E$308.2; no longer E$103.E
- net S$83: now also E$208.E, E$209.E, E$217.A, E$218.A, E$224.E, E$225.E, E$233.A, E$234.A, E$275.1, E$301.1, E$306.1, E$308.1; no longer E$106.E
- net S$84: now also E$216.A, E$217.C; no longer E$104.C, E$106.B, E$117.1
- net S$85: now also E$215.A, E$218.C; no longer E$105.B, E$115.2
- net S$86: now also E$223.C, E$226.C, E$231.C, E$232.C, E$236.2, E$237.2, E$274.1, E$309.C; no longer E$104.B, E$118.2
- net S$87: now also E$238.1, E$271.1; no longer E$112.A, E$113.C
- net S$90: now also E$310.B, E$312.C, E$323.1; no longer E$104.E, E$105.E, E$113.A, E$114.A
- net S$91: now also E$310.E; no longer E$115.1
- net S$94: now also E$312.B, E$322.2; no longer E$120.B, E$122.C, E$133.1
- net S$95: now also E$311.B, E$325.2; no longer E$120.E
- net S$98: now also E$326.B, E$328.C, E$339.1; no longer E$122.B, E$132.2
- net S$99: now also E$326.E; no longer E$121.B, E$135.2
Routing:
- net S$228: track 3.81 -> 297.8 mm
- net S$112: track 5.08 -> 297.8 mm
- net S$199: track 8.67 -> 297.8 mm
- net S$83: track 8.67 -> 297.8 mm
- net S$170: track 19.6 -> 297.8 mm, vias 1 -> 0
- net S$141: track 65.8 -> 297.8 mm
- net S$140: track 2.54 -> 134.6 mm
- net S$111: track 3.81 -> 134.6 mm
- net S$82: track 8.67 -> 134.6 mm
- net S$227: track 18.8 -> 134.6 mm
- net S$198: track 18.8 -> 134.6 mm
- net S$246: track 90.4 -> 0.00 mm, vias 1 -> 0
- net S$298: track 90.4 -> 0.00 mm, vias 1 -> 0
- net S$272: track 90.4 -> 0.00 mm, vias 1 -> 0
- net S$23: track 90.4 -> 0.00 mm, vias 1 -> 0
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- added copper zone on layer 16, net S$109
- added copper zone on layer 16, net S$138
- added copper zone on layer 16, net S$167
- added copper zone on layer 16, net S$196
- added copper zone on layer 16, net S$225
- added copper zone on layer 16, net S$80
Other:
- board text added: "Made in Hungary by Zoltán Farkas."
