File: microcap/pcb/tmp.brd (EAGLE design)
At the start: 618 parts

Commit message: pcb update
Parts:
- removed E$619, E$620, E$621, E$622, E$635, E$636, E$637, E$638, E$722, E$723, E$724, E$725, E$738, E$739, E$740, E$741: (no value), transistor:TO92-CBE
- removed E$623, E$624, E$625, E$626, E$639, E$640, E$641, E$642, E$726, E$727, E$728, E$729, E$742, E$743, E$744, E$745: (no value), transistor:T-30_V
- removed E$627, E$628, E$629, E$630, E$643, E$644, E$645, E$646, E$730, E$731, E$732, E$733, E$746, E$747, E$748, E$749: (no value), diode:C2992
- removed E$631, E$632, E$633, E$634, E$647, E$648, E$649, E$650, E$717, E$719, E$734, E$735, E$736, E$737, E$750, E$751, E$752, E$753, E$820, E$822: (no value), resistor:0207/10
- removed E$651, E$652, E$653, E$654, E$655, E$656, E$657, E$658, E$659, E$660, E$661, E$662, E$663, E$664, E$665, E$666, E$667, E$668, E$669, E$670, E$671, E$672, E$673, E$674, E$675, E$676, E$677, E$678, E$679, E$680, E$681, E$682, E$683, E$684, E$685, E$686, E$687, E$688, E$689, E$690, E$691, E$692, E$693, E$694, E$695, E$696, E$697, E$698, E$699, E$700, E$701, E$702, E$703, E$704, E$705, E$706, E$707, E$708, E$709, E$710, E$711, E$712, E$713, E$714, E$715, E$716, E$754, E$755, E$756, E$757, E$758, E$759, E$760, E$761, E$762, E$763, E$764, E$765, E$766, E$767, E$768, E$769, E$770, E$771, E$772, E$773, E$774, E$775, E$776, E$777, E$778, E$779, E$780, E$781, E$782, E$783, E$784, E$785, E$786, E$787, E$788, E$789, E$790, E$791, E$792, E$793, E$794, E$795, E$796, E$797, E$798, E$799, E$800, E$801, E$802, E$803, E$804, E$805, E$806, E$807, E$808, E$809, E$810, E$811, E$812, E$813, E$814, E$815, E$816, E$817, E$818, E$819: (no value), pinhead:1X01
- removed E$718, E$821: (no value), capacitor-wima:C5B2.5
- removed E$720, E$823: (no value), capacitor-wima:C2.5-2
- removed E$721, E$824: (no value), diode:ZDIO-10
- added E$1, E$103, E$104, E$106, E$107, E$120, E$121, E$122, E$123, E$2, E$3, E$4, E$5, E$6, E$7, E$8: (no value), transistor:TO92-CBE
- added E$10, E$100, E$11, E$136, E$137, E$138, E$139, E$140, E$141, E$142, E$143, E$144, E$145, E$146, E$147, E$148, E$149, E$150, E$151, E$152, E$153, E$154, E$155, E$156, E$157, E$158, E$159, E$160, E$161, E$162, E$163, E$164, E$165, E$166, E$167, E$168, E$169, E$170, E$171, E$172, E$173, E$174, E$175, E$176, E$177, E$178, E$179, E$180, E$181, E$182, E$183, E$184, E$185, E$186, E$187, E$188, E$189, E$190, E$191, E$192, E$193, E$194, E$195, E$196, E$197, E$198, E$199, E$200, E$201, E$24, E$25, E$26, E$27, E$28, E$29, E$30, E$31, E$32, E$33, E$34, E$35, E$36, E$37, E$38, E$39, E$52, E$53, E$54, E$55, E$56, E$57, E$58, E$59, E$60, E$61, E$62, E$63, E$64, E$65, E$66, E$67, E$68, E$69, E$70, E$71, E$72, E$73, E$74, E$75, E$76, E$77, E$78, E$79, E$80, E$81, E$82, E$83, E$84, E$85, E$86, E$87, E$88, E$89, E$9, E$90, E$91, E$92, E$95, E$96, E$97, E$98, E$99: (no value), pinhead:1X01
- added E$101, E$203: (no value), capacitor-wima:C5B2.5
- added E$102, E$205: (no value), capacitor-wima:C2.5-2
- added E$105, E$206: (no value), diode:ZDIO-10
- added E$108, E$109, E$110, E$111, E$12, E$124, E$125, E$126, E$127, E$13, E$14, E$15, E$40, E$41, E$42, E$43: (no value), transistor:T-30_V
- added E$112, E$113, E$114, E$115, E$128, E$129, E$130, E$131, E$16, E$17, E$18, E$19, E$44, E$45, E$46, E$47: (no value), diode:C2992
- added E$116, E$117, E$118, E$119, E$132, E$133, E$134, E$135, E$20, E$202, E$204, E$21, E$22, E$23, E$48, E$49, E$50, E$51, E$93, E$94: (no value), resistor:0207/10
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Connections:
- removed net S$105: E$334.A, E$337.C
- removed net S$123: E$415.B, E$425.2
- removed net S$124: E$414.B, E$428.2
- removed net S$134: E$437.A, E$440.C
- removed net S$152: E$518.B, E$528.2
- removed net S$153: E$517.B, E$531.2
- removed net S$163: E$540.A, E$543.C
- removed net S$177: E$619.B, E$621.C, E$632.1
- removed net S$178: E$619.E
- removed net S$179: E$622.E
- removed net S$180: E$620.C, E$622.B, E$633.1
- removed net S$181: E$621.B, E$631.2
- removed net S$182: E$620.B, E$634.2
- removed net S$185: E$635.B, E$637.C, E$648.1
- removed net S$186: E$635.E
- removed net S$187: E$638.E
- removed net S$188: E$636.C, E$638.B, E$649.1
- removed net S$189: E$636.B, E$650.2
- removed net S$190: E$637.B, E$647.2
- removed net S$191: E$644.A, E$645.C
- removed net S$192: E$643.A, E$646.C
- removed net S$193: E$647.1, E$682.1
- removed net S$194: E$634.1, E$680.1
- removed net S$195: E$631.1, E$681.1
- removed net S$197: E$694.1
- removed net S$198: E$619.C, E$622.C, E$627.C, E$628.C, E$632.2, E$633.2, E$656.1, E$671.1, E$672.1, E$718.2, E$720.2
- removed net S$199: E$620.E, E$621.E, E$629.A, E$630.A, E$636.E, E$637.E, E$645.A, E$646.A, E$687.1, E$713.1, E$718.1, E$720.1
- removed net S$200: E$628.A, E$629.C
- removed net S$201: E$627.A, E$630.C
- removed net S$202: E$635.C, E$638.C, E$643.C, E$644.C, E$648.2, E$649.2, E$686.1, E$721.C
- removed net S$203: E$650.1, E$683.1
- removed net S$206: E$722.B, E$724.C, E$735.1
- removed net S$207: E$722.E
- removed net S$208: E$725.E
- removed net S$209: E$723.C, E$725.B, E$736.1
- removed net S$210: E$724.B, E$734.2
- removed net S$211: E$723.B, E$737.2
- removed net S$214: E$738.B, E$740.C, E$751.1
- removed net S$215: E$738.E
- removed net S$216: E$741.E
- removed net S$217: E$739.C, E$741.B, E$752.1
- removed net S$218: E$739.B, E$753.2
- removed net S$219: E$740.B, E$750.2
- removed net S$220: E$747.A, E$748.C
- removed net S$221: E$746.A, E$749.C
- removed net S$222: E$750.1, E$785.1
- removed net S$223: E$737.1, E$783.1
- removed net S$224: E$734.1, E$784.1
- removed net S$226: E$797.1
- removed net S$227: E$722.C, E$725.C, E$730.C, E$731.C, E$735.2, E$736.2, E$759.1, E$774.1, E$775.1, E$821.2, E$823.2
- removed net S$228: E$723.E, E$724.E, E$732.A, E$733.A, E$739.E, E$740.E, E$748.A, E$749.A, E$790.1, E$816.1, E$821.1, E$823.1
- removed net S$229: E$731.A, E$732.C
- removed net S$230: E$730.A, E$733.C
- removed net S$231: E$738.C, E$741.C, E$746.C, E$747.C, E$751.2, E$752.2, E$789.1, E$824.C
- removed net S$232: E$753.1, E$786.1
- removed net S$65: E$209.B, E$219.2
- removed net S$66: E$208.B, E$222.2
- removed net S$76: E$231.A, E$234.C
- removed net S$94: E$312.B, E$322.2
- removed net S$95: E$311.B, E$325.2
- new net S$10: E$1.E
- new net S$109: E$319.A, E$320.C
- new net S$11: E$5.E
- new net S$12: E$17.A, E$18.C
- new net S$125: E$429.B, E$431.C, E$442.1
- new net S$126: E$429.E
- new net S$138: E$422.A, E$423.C
- new net S$14: E$8.E
- new net S$15: E$23.1, E$67.1
- new net S$154: E$532.B, E$534.C, E$545.1
- new net S$155: E$532.E
- new net S$16: E$22.1, E$6.C, E$8.B
- new net S$167: E$525.A, E$526.C
- new net S$17: E$23.2, E$6.B
- new net S$18: E$51.1, E$64.1
- new net S$19: E$16.A, E$19.C
- new net S$2: E$2.C, E$4.B, E$50.1
- new net S$20: E$101.1, E$102.1, E$18.A, E$19.A, E$2.E, E$3.E, E$46.A, E$47.A, E$6.E, E$7.E, E$71.1, E$97.1
- new net S$21: E$20.2, E$7.B
- new net S$22: E$44.A, E$47.C
- new net S$23: E$48.1, E$65.1
- new net S$25: E$1.C, E$101.2, E$102.2, E$29.1, E$4.C, E$44.C, E$45.C, E$49.2, E$50.2, E$58.1, E$59.1
- new net S$26: E$77.1
- new net S$28: E$105.C, E$16.C, E$17.C, E$21.2, E$22.2, E$5.C, E$70.1, E$8.C
- new net S$31: E$103.B, E$106.C, E$117.1
- new net S$32: E$103.E
- new net S$33: E$107.E
- new net S$34: E$104.C, E$107.B, E$118.1
- new net S$36: E$20.1, E$66.1
- new net S$38: E$120.B, E$122.C, E$133.1
- new net S$39: E$120.E
- new net S$4: E$4.E
- new net S$40: E$123.E
- new net S$41: E$121.C, E$123.B, E$134.1
- new net S$42: E$129.A, E$130.C
- new net S$43: E$128.A, E$131.C
- new net S$44: E$132.1, E$167.1
- new net S$45: E$119.1, E$165.1
- new net S$46: E$116.1, E$166.1
- new net S$48: E$179.1
- new net S$49: E$103.C, E$107.C, E$112.C, E$113.C, E$117.2, E$118.2, E$141.1, E$156.1, E$157.1, E$203.2, E$205.2
- new net S$5: E$3.B, E$48.2
- new net S$50: E$104.E, E$106.E, E$114.A, E$115.A, E$121.E, E$122.E, E$130.A, E$131.A, E$172.1, E$198.1, E$203.1, E$205.1
- new net S$51: E$113.A, E$114.C
- new net S$52: E$112.A, E$115.C
- new net S$53: E$120.C, E$123.C, E$128.C, E$129.C, E$133.2, E$134.2, E$171.1, E$206.C
- new net S$54: E$135.1, E$168.1
- new net S$55: E$106.B, E$116.2
- new net S$56: E$104.B, E$119.2
- new net S$57: E$121.B, E$135.2
- new net S$58: E$122.B, E$132.2
- new net S$6: E$2.B, E$51.2
- new net S$67: E$223.B, E$225.C, E$236.1
- new net S$68: E$223.E
- new net S$7: E$21.1, E$5.B, E$7.C
- new net S$8: E$45.A, E$46.C
- new net S$80: E$216.A, E$217.C
- new net S$9: E$1.B, E$3.C, E$49.1
- new net S$96: E$326.B, E$328.C, E$339.1
- new net S$97: E$326.E
- net S$100: now also E$335.A, E$336.C; no longer E$329.E
- net S$101: now also E$334.A, E$337.C; no longer E$327.C, E$329.B, E$340.1
- net S$102: now also E$338.1, E$373.1; no longer E$327.B, E$341.2
- net S$103: now also E$325.1, E$371.1; no longer E$328.B, E$338.2
- net S$104: now also E$322.1, E$372.1; no longer E$335.A, E$336.C
- net S$106: now also E$385.1; no longer E$338.1, E$373.1
- net S$107: now also E$310.C, E$313.C, E$318.C, E$319.C, E$323.2, E$324.2, E$347.1, E$362.1, E$363.1, E$409.2, E$411.2; no longer E$325.1, E$371.1
- net S$108: now also E$311.E, E$312.E, E$320.A, E$321.A, E$327.E, E$328.E, E$336.A, E$337.A, E$378.1, E$404.1, E$409.1, E$411.1; no longer E$322.1, E$372.1
- net S$110: now also E$318.A, E$321.C; no longer E$385.1
- net S$111: now also E$326.C, E$329.C, E$334.C, E$335.C, E$339.2, E$340.2, E$377.1, E$412.C; no longer E$310.C, E$313.C, E$318.C, E$319.C, E$323.2, E$324.2, E$347.1, E$362.1, E$363.1, E$409.2, E$411.2
- net S$112: now also E$341.1, E$374.1; no longer E$311.E, E$312.E, E$320.A, E$321.A, E$327.E, E$328.E, E$336.A, E$337.A, E$378.1, E$404.1, E$409.1, E$411.1
- net S$113: now also E$312.B, E$322.2; no longer E$319.A, E$320.C
- net S$114: now also E$311.B, E$325.2; no longer E$318.A, E$321.C
- net S$115: now also E$327.B, E$341.2; no longer E$326.C, E$329.C, E$334.C, E$335.C, E$339.2, E$340.2, E$377.1, E$412.C
- net S$116: now also E$328.B, E$338.2; no longer E$341.1, E$374.1
- net S$127: now also E$432.E; no longer E$429.B, E$431.C, E$442.1
- net S$128: now also E$430.C, E$432.B, E$443.1; no longer E$429.E
- net S$129: now also E$438.A, E$439.C; no longer E$432.E
- net S$130: now also E$437.A, E$440.C; no longer E$430.C, E$432.B, E$443.1
- net S$131: now also E$441.1, E$476.1; no longer E$430.B, E$444.2
- net S$132: now also E$428.1, E$474.1; no longer E$431.B, E$441.2
- net S$133: now also E$425.1, E$475.1; no longer E$438.A, E$439.C
- net S$135: now also E$488.1; no longer E$441.1, E$476.1
- net S$136: now also E$413.C, E$416.C, E$421.C, E$422.C, E$426.2, E$427.2, E$450.1, E$465.1, E$466.1, E$512.2, E$514.2; no longer E$428.1, E$474.1
- net S$137: now also E$414.E, E$415.E, E$423.A, E$424.A, E$430.E, E$431.E, E$439.A, E$440.A, E$481.1, E$507.1, E$512.1, E$514.1; no longer E$425.1, E$475.1
- net S$139: now also E$421.A, E$424.C; no longer E$488.1
- net S$140: now also E$429.C, E$432.C, E$437.C, E$438.C, E$442.2, E$443.2, E$480.1, E$515.C; no longer E$413.C, E$416.C, E$421.C, E$422.C, E$426.2, E$427.2, E$450.1, E$465.1, E$466.1, E$512.2, E$514.2
- net S$141: now also E$444.1, E$477.1; no longer E$414.E, E$415.E, E$423.A, E$424.A, E$430.E, E$431.E, E$439.A, E$440.A, E$481.1, E$507.1, E$512.1, E$514.1
- net S$142: now also E$415.B, E$425.2; no longer E$422.A, E$423.C
- net S$143: now also E$414.B, E$428.2; no longer E$421.A, E$424.C
- net S$144: now also E$430.B, E$444.2; no longer E$429.C, E$432.C, E$437.C, E$438.C, E$442.2, E$443.2, E$480.1, E$515.C
- net S$145: now also E$431.B, E$441.2; no longer E$444.1, E$477.1
- net S$156: now also E$535.E; no longer E$532.B, E$534.C, E$545.1
- net S$157: now also E$533.C, E$535.B, E$546.1; no longer E$532.E
- net S$158: now also E$541.A, E$542.C; no longer E$535.E
- net S$159: now also E$540.A, E$543.C; no longer E$533.C, E$535.B, E$546.1
- net S$160: now also E$544.1, E$579.1; no longer E$533.B, E$547.2
- net S$161: now also E$531.1, E$577.1; no longer E$534.B, E$544.2
- net S$162: now also E$528.1, E$578.1; no longer E$541.A, E$542.C
- net S$164: now also E$591.1; no longer E$544.1, E$579.1
- net S$165: now also E$516.C, E$519.C, E$524.C, E$525.C, E$529.2, E$530.2, E$553.1, E$568.1, E$569.1, E$615.2, E$617.2; no longer E$531.1, E$577.1
- net S$166: now also E$517.E, E$518.E, E$526.A, E$527.A, E$533.E, E$534.E, E$542.A, E$543.A, E$584.1, E$610.1, E$615.1, E$617.1; no longer E$528.1, E$578.1
- net S$168: now also E$524.A, E$527.C; no longer E$591.1
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Routing:
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- added copper zone on layer 16, net S$105
- added copper zone on layer 16, net S$134
- added copper zone on layer 16, net S$163
- added copper zone on layer 16, net S$24
- added copper zone on layer 16, net S$47
- added copper zone on layer 16, net S$76
- removed copper zone on layer 16, net S$109
- removed copper zone on layer 16, net S$138
- removed copper zone on layer 16, net S$167
- removed copper zone on layer 16, net S$196
- removed copper zone on layer 16, net S$225
- removed copper zone on layer 16, net S$80

Commit message: pcb update
Parts:
- added E$619, E$621: (no value), resistor:0207/10
- added E$620: (no value), capacitor-wima:C5B2.5
- added E$622: (no value), capacitor-wima:C2.5-2
- added E$623: (no value), diode:ZDIO-10
- added E$624: (no value), switch:255SB
- E$103, E$208, E$312, E$416: device transistor:TO92-CBE -> switch:255SB
- E$108, E$124, E$211, E$212, E$227, E$228, E$314, E$315, E$316, E$330, E$331, E$332, E$417, E$418, E$419, E$420, E$433, E$434, E$435, E$436, E$521, E$522, E$523, E$537, E$538, E$539: device transistor:T-30_V -> transistor:TO92-CBE
- E$112, E$128, E$215, E$216, E$231, E$232, E$318, E$319, E$320, E$334, E$335, E$336, E$421, E$422, E$423, E$424, E$437, E$438, E$439, E$440, E$525, E$526, E$527, E$541, E$542, E$543: device diode:C2992 -> transistor:T-30_V
- E$116, E$132, E$219, E$220, E$235, E$236, E$322, E$323, E$324, E$338, E$339, E$340, E$425, E$426, E$427, E$428, E$441, E$442, E$443, E$444, E$529, E$530, E$531, E$545, E$546, E$547: device resistor:0207/10 -> diode:C2992
- E$120, E$223, E$224, E$326, E$327, E$328, E$413, E$429, E$430, E$431, E$432, E$517, E$533, E$534, E$535: device transistor:TO92-CBE -> resistor:0207/10
- E$136, E$239, E$240, E$342, E$343, E$344, E$445, E$446, E$447, E$448, E$549, E$550, E$551, E$552: device pinhead:1X01 -> resistor:0207/10
- E$202, E$305, E$408, E$410, E$511, E$513, E$614, E$616: device resistor:0207/10 -> pinhead:1X01
- E$203: device capacitor-wima:C5B2.5 -> resistor:0207/10
- E$204: device resistor:0207/10 -> capacitor-wima:C5B2.5
- E$205, E$411: device capacitor-wima:C2.5-2 -> resistor:0207/10
- E$206: device diode:ZDIO-10 -> capacitor-wima:C2.5-2
- E$207, E$311, E$415, E$519: device transistor:TO92-CBE -> diode:ZDIO-10
- E$306, E$409, E$512, E$615: device capacitor-wima:C5B2.5 -> pinhead:1X01
- E$308: device capacitor-wima:C2.5-2 -> capacitor-wima:C5B2.5
- E$309, E$515: device diode:ZDIO-10 -> resistor:0207/10
- E$310, E$414, E$518: device transistor:TO92-CBE -> capacitor-wima:C2.5-2
- E$412: device diode:ZDIO-10 -> capacitor-wima:C5B2.5
- E$514, E$617: device capacitor-wima:C2.5-2 -> pinhead:1X01
- E$516: device transistor:TO92-CBE -> capacitor-wima:C5B2.5
- E$520: device transistor:T-30_V -> switch:255SB
- E$524, E$540: device diode:C2992 -> transistor:TO92-CBE
- E$528, E$544: device resistor:0207/10 -> transistor:T-30_V
- E$532: device transistor:TO92-CBE -> diode:C2992
- E$536: device transistor:T-30_V -> resistor:0207/10
- E$548: device pinhead:1X01 -> diode:C2992
- E$618: device diode:ZDIO-10 -> pinhead:1X01
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Connections:
- removed net S$20: E$101.1, E$102.1, E$18.A, E$19.A, E$2.E, E$3.E, E$46.A, E$47.A, E$6.E, E$7.E, E$71.1, E$97.1
- new net S$29: E$1.C, E$101.2, E$102.2, E$103.2, E$29.1, E$4.C, E$44.C, E$45.C, E$49.2, E$50.2, E$58.1, E$59.1
- net S$100: now also E$338.A, E$339.C; no longer E$335.A, E$336.C
- net S$101: now also E$337.A, E$340.C; no longer E$334.A, E$337.C
- net S$102: now also E$341.1, E$376.1; no longer E$338.1, E$373.1
- net S$103: now also E$328.1, E$374.1; no longer E$325.1, E$371.1
- net S$104: now also E$325.1, E$375.1; no longer E$322.1, E$372.1
- net S$106: now also E$388.1; no longer E$385.1
- net S$107: now also E$322.A, E$323.C; no longer E$310.C, E$313.C, E$318.C, E$319.C, E$323.2, E$324.2, E$347.1, E$362.1, E$363.1, E$409.2, E$411.2
- net S$108: now also E$324.C; no longer E$311.E, E$312.E, E$320.A, E$327.E, E$328.E, E$336.A, E$337.A, E$378.1, E$404.1, E$409.1, E$411.1
- net S$109: now also E$329.C, E$332.C, E$337.C, E$338.C, E$342.2, E$343.2, E$380.1, E$415.C; no longer E$319.A, E$320.C
- net S$110: now also E$344.1, E$377.1; no longer E$318.A, E$321.C
- net S$111: now also E$315.B, E$325.2; no longer E$326.C, E$329.C, E$334.C, E$335.C, E$339.2, E$340.2, E$377.1, E$412.C
- net S$112: now also E$314.B, E$328.2; no longer E$341.1, E$374.1
- net S$113: now also E$330.B, E$344.2; no longer E$312.B, E$322.2
- net S$114: now also E$331.B, E$341.2; no longer E$311.B, E$325.2
- net S$115: now also E$313.C, E$316.C, E$321.C, E$322.C, E$326.2, E$327.2, E$350.1, E$365.1, E$366.1, E$412.2, E$414.2, E$416.2; no longer E$327.B, E$341.2
- net S$116: now also E$314.E, E$315.E, E$323.A, E$324.A, E$330.E, E$331.E, E$339.A, E$340.A, E$381.1, E$407.1, E$412.1, E$414.1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; no longer E$328.B, E$338.2
- net S$119: now also E$417.B, E$419.C, E$430.1; no longer E$413.B, E$415.C, E$426.1
- net S$120: now also E$417.E; no longer E$413.E
- net S$121: now also E$420.E; no longer E$416.E
- net S$122: now also E$418.C, E$420.B, E$431.1; no longer E$414.C, E$416.B, E$427.1
- net S$125: now also E$433.B, E$435.C, E$446.1; no longer E$429.B, E$431.C, E$442.1
- net S$126: now also E$433.E; no longer E$429.E
- net S$127: now also E$436.E; no longer E$432.E
- net S$128: now also E$434.C, E$436.B, E$447.1; no longer E$430.C, E$432.B, E$443.1
- net S$129: now also E$442.A, E$443.C; no longer E$438.A, E$439.C
- net S$130: now also E$441.A, E$444.C; no longer E$437.A, E$440.C
- net S$131: now also E$445.1, E$480.1; no longer E$441.1, E$476.1
- net S$132: now also E$432.1, E$478.1; no longer E$428.1, E$474.1
- net S$133: now also E$429.1, E$479.1; no longer E$425.1, E$475.1
- net S$135: now also E$492.1; no longer E$488.1
- net S$136: now also E$426.A, E$427.C; no longer E$413.C, E$416.C, E$421.C, E$422.C, E$426.2, E$427.2, E$450.1, E$465.1, E$466.1, E$512.2, E$514.2
- net S$137: now also E$425.A, E$428.C; no longer E$414.E, E$415.E, E$423.A, E$424.A, E$430.E, E$431.E, E$439.A, E$440.A, E$481.1, E$507.1, E$512.1, E$514.1
- net S$138: now also E$433.C, E$436.C, E$441.C, E$442.C, E$446.2, E$447.2, E$484.1, E$519.C; no longer E$422.A, E$423.C
- net S$139: now also E$448.1, E$481.1; no longer E$421.A, E$424.C
- net S$140: now also E$419.B, E$429.2; no longer E$429.C, E$432.C, E$437.C, E$438.C, E$442.2, E$443.2, E$480.1, E$515.C
- net S$141: now also E$418.B, E$432.2; no longer E$444.1, E$477.1
- net S$142: now also E$434.B, E$448.2; no longer E$415.B, E$425.2
- net S$143: now also E$435.B, E$445.2; no longer E$414.B, E$428.2
- net S$144: now also E$417.C, E$420.C, E$425.C, E$426.C, E$430.2, E$431.2, E$454.1, E$469.1, E$470.1, E$516.2, E$518.2, E$520.2; no longer E$430.B, E$444.2
- net S$145: now also E$418.E, E$419.E, E$427.A, E$428.A, E$434.E, E$435.E, E$443.A, E$444.A, E$485.1, E$511.1, E$516.1, E$518.1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; no longer E$431.B, E$441.2
- net S$148: now also E$521.B, E$523.C, E$534.1; no longer E$516.B, E$518.C, E$529.1
- net S$149: now also E$521.E; no longer E$516.E
- net S$150: now also E$524.E; no longer E$519.E
- net S$151: now also E$522.C, E$524.B, E$535.1; no longer E$517.C, E$519.B, E$530.1
- net S$154: now also E$537.B, E$539.C, E$550.1; no longer E$532.B, E$534.C, E$545.1
- net S$155: now also E$537.E; no longer E$532.E
- net S$156: now also E$540.E; no longer E$535.E
- net S$157: now also E$538.C, E$540.B, E$551.1; no longer E$533.C, E$535.B, E$546.1
- net S$158: now also E$546.A, E$547.C; no longer E$541.A, E$542.C
- net S$159: now also E$545.A, E$548.C; no longer E$540.A, E$543.C
- net S$160: now also E$549.1, E$584.1; no longer E$544.1, E$579.1
- net S$161: now also E$536.1, E$582.1; no longer E$531.1, E$577.1
- net S$162: now also E$533.1, E$583.1; no longer E$528.1, E$578.1
- net S$164: now also E$596.1; no longer E$591.1
- net S$165: now also E$530.A, E$531.C; no longer E$516.C, E$519.C, E$524.C, E$525.C, E$529.2, E$530.2, E$553.1, E$568.1, E$569.1, E$615.2, E$617.2
- net S$166: now also E$529.A, E$532.C; no longer E$517.E, E$518.E, E$526.A, E$527.A, E$533.E, E$534.E, E$542.A, E$543.A, E$584.1, E$610.1, E$615.1, E$617.1
- net S$167: now also E$537.C, E$540.C, E$545.C, E$546.C, E$550.2, E$551.2, E$588.1, E$623.C; no longer E$525.A, E$526.C
- net S$168: now also E$552.1, E$585.1; no longer E$524.A, E$527.C
- net S$169: now also E$523.B, E$533.2; no longer E$532.C, E$535.C, E$540.C, E$541.C, E$545.2, E$546.2, E$583.1, E$618.C
- net S$170: now also E$522.B, E$536.2; no longer E$547.1, E$580.1
- net S$171: now also E$538.B, E$552.2; no longer E$518.B, E$528.2
- net S$172: now also E$539.B, E$549.2; no longer E$517.B, E$531.2
- net S$173: now also E$521.C, E$524.C, E$529.C, E$530.C, E$534.2, E$535.2, E$558.1, E$573.1, E$574.1, E$620.2, E$622.2, E$624.2; no longer E$533.B, E$547.2
- net S$174: now also E$522.E, E$523.E, E$531.A, E$532.A, E$538.E, E$539.E, E$547.A, E$548.A, E$589.1, E$615.1, E$620.1, E$622.1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; no longer E$534.B, E$544.2
- net S$25: now also E$101.1, E$102.1, E$103.1, E$18.A, E$19.A, E$2.E, E$3.E, E$46.A, E$47.A, E$6.E, E$7.E, E$71.1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; no longer E$1.C, E$101.2, E$102.2, E$29.1, E$4.C, E$44.C, E$45.C, E$49.2, E$50.2, E$58.1, E$59.1
- net S$31: now also E$104.B, E$107.C, E$118.1; no longer E$103.B, E$106.C, E$117.1
- net S$32: now also E$104.E; no longer E$103.E
- net S$33: now also E$108.E; no longer E$107.E
- net S$34: now also E$106.C, E$108.B, E$119.1; no longer E$104.C, E$107.B, E$118.1
- net S$38: now also E$121.B, E$123.C, E$134.1; no longer E$120.B, E$122.C, E$133.1
- net S$39: now also E$121.E; no longer E$120.E
- net S$40: now also E$124.E; no longer E$123.E
- net S$41: now also E$122.C, E$124.B, E$135.1; no longer E$121.C, E$123.B, E$134.1
- net S$42: now also E$130.A, E$131.C; no longer E$129.A, E$130.C
- net S$43: now also E$129.A, E$132.C; no longer E$128.A, E$131.C
- net S$44: now also E$133.1, E$168.1; no longer E$132.1, E$167.1
- net S$45: now also E$120.1, E$166.1; no longer E$119.1, E$165.1
- net S$46: now also E$117.1, E$167.1; no longer E$116.1, E$166.1
- net S$48: now also E$180.1; no longer E$179.1
- net S$49: now also E$114.A, E$115.C; no longer E$103.C, E$107.C, E$112.C, E$113.C, E$117.2, E$118.2, E$141.1, E$156.1, E$157.1, E$203.2, E$205.2
- net S$50: now also E$113.A, E$116.C; no longer E$104.E, E$106.E, E$114.A, E$115.A, E$121.E, E$122.E, E$130.A, E$131.A, E$172.1, E$198.1, E$203.1, E$205.1
- net S$51: now also E$121.C, E$124.C, E$129.C, E$130.C, E$134.2, E$135.2, E$172.1, E$207.C; no longer E$113.A, E$114.C
- net S$52: now also E$136.1, E$169.1; no longer E$112.A, E$115.C
- net S$53: now also E$107.B, E$117.2; no longer E$120.C, E$123.C, E$128.C, E$129.C, E$133.2, E$134.2, E$171.1, E$206.C
- net S$54: now also E$106.B, E$120.2; no longer E$135.1, E$168.1
- net S$55: now also E$122.B, E$136.2; no longer E$106.B, E$116.2
- net S$56: now also E$123.B, E$133.2; no longer E$104.B, E$119.2
- net S$57: now also E$104.C, E$108.C, E$113.C, E$114.C, E$118.2, E$119.2, E$142.1, E$157.1, E$158.1, E$204.2, E$206.2, E$208.2; no longer E$121.B, E$135.2
- net S$58: now also E$106.E, E$107.E, E$115.A, E$116.A, E$122.E, E$123.E, E$131.A, E$132.A, E$173.1, E$199.1, E$204.1, E$206.1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; no longer E$122.B, E$132.2
- net S$61: now also E$209.B, E$211.C, E$222.1; no longer E$207.B, E$209.C, E$220.1
- net S$62: now also E$209.E; no longer E$207.E
- net S$63: now also E$212.E; no longer E$210.E
- net S$64: now also E$210.C, E$212.B, E$223.1; no longer E$208.C, E$210.B, E$221.1
- net S$67: now also E$225.B, E$227.C, E$238.1; no longer E$223.B, E$225.C, E$236.1
- net S$68: now also E$225.E; no longer E$223.E
- net S$69: now also E$228.E; no longer E$226.E
- net S$70: now also E$226.C, E$228.B, E$239.1; no longer E$224.C, E$226.B, E$237.1
- net S$71: now also E$234.A, E$235.C; no longer E$232.A, E$233.C
- net S$72: now also E$233.A, E$236.C; no longer E$231.A, E$234.C
- net S$73: now also E$237.1, E$272.1; no longer E$235.1, E$270.1
- net S$74: now also E$224.1, E$270.1; no longer E$222.1, E$268.1
- net S$75: now also E$221.1, E$271.1; no longer E$219.1, E$269.1
- net S$77: now also E$284.1; no longer E$282.1
- net S$78: now also E$218.A, E$219.C; no longer E$207.C, E$210.C, E$215.C, E$216.C, E$220.2, E$221.2, E$244.1, E$259.1, E$260.1, E$306.2, E$308.2
- net S$79: now also E$220.C; no longer E$208.E, E$209.E, E$218.A, E$224.E, E$225.E, E$233.A, E$234.A, E$275.1, E$301.1, E$306.1, E$308.1
- net S$80: now also E$225.C, E$228.C, E$233.C, E$234.C, E$238.2, E$239.2, E$276.1, E$311.C; no longer E$216.A, E$217.C
- net S$81: now also E$240.1, E$273.1; no longer E$215.A, E$218.C
- net S$82: now also E$211.B, E$221.2; no longer E$223.C, E$226.C, E$231.C, E$232.C, E$236.2, E$237.2, E$274.1, E$309.C
- net S$83: now also E$210.B, E$224.2; no longer E$238.1, E$271.1
- net S$84: now also E$226.B, E$240.2; no longer E$209.B, E$219.2
- net S$85: now also E$227.B, E$237.2; no longer E$208.B, E$222.2
- net S$86: now also E$209.C, E$212.C, E$217.C, E$218.C, E$222.2, E$223.2, E$246.1, E$261.1, E$262.1, E$308.2, E$310.2, E$312.2; no longer E$224.B, E$238.2
- net S$87: now also E$210.E, E$211.E, E$219.A, E$220.A, E$226.E, E$227.E, E$235.A, E$236.A, E$277.1, E$303.1, E$308.1, E$310.1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; no longer E$225.B, E$235.2
- net S$90: now also E$313.B, E$315.C, E$326.1; no longer E$310.B, E$312.C, E$323.1
- net S$91: now also E$313.E; no longer E$310.E
- net S$92: now also E$316.E; no longer E$313.E
- net S$93: now also E$314.C, E$316.B, E$327.1; no longer E$311.C, E$313.B, E$324.1
- net S$96: now also E$329.B, E$331.C, E$342.1; no longer E$326.B, E$328.C, E$339.1
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Routing:
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
Commit message: pcb update
Parts:
- moved E$10 29.2 mm to (111.8, 52.1)
- moved E$100 29.2 mm to (111.8, 80.0)
- moved E$101 29.2 mm to (97.8, 87.6)
- moved E$105 29.2 mm to (88.9, 55.9)
- moved E$107 29.2 mm to (134.6, 81.3)
- moved E$108 29.2 mm to (166.4, 92.7)
- moved E$109 29.2 mm to (163.8, 92.7)
- moved E$110 29.2 mm to (144.8, 81.3)
- moved E$111 29.2 mm to (148.6, 92.7)
- moved E$117 29.2 mm to (130.8, 74.9)
- moved E$118 29.2 mm to (134.6, 91.4)
- moved E$123 29.2 mm to (134.6, 45.7)
- moved E$124 29.2 mm to (166.4, 57.1)
- moved E$125 29.2 mm to (163.8, 57.1)
- moved E$126 29.2 mm to (144.8, 45.7)
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Connections:
- removed net S$29: E$1.C, E$101.2, E$102.2, E$103.2, E$29.1, E$4.C, E$44.C, E$45.C, E$49.2, E$50.2, E$58.1, E$59.1
- new net S$20: E$1.C, E$101.2, E$102.2, E$103.1, E$29.1, E$4.C, E$44.C, E$45.C, E$49.2, E$50.2, E$58.1, E$59.1
- net S$115: now also E$416.1; no longer E$416.2
- net S$116: no longer E$416.1
- net S$144: now also E$520.1; no longer E$520.2
- net S$145: no longer E$520.1
- net S$173: now also E$624.1; no longer E$624.2
- net S$174: no longer E$624.1
- net S$25: no longer E$103.1
- net S$57: now also E$208.1; no longer E$208.2
- net S$58: no longer E$208.1
- net S$86: now also E$312.1; no longer E$312.2
- net S$87: no longer E$312.1
Routing:
- net S$29: track 156.0 -> 19.6 mm
- net S$20: track 19.6 -> 151.4 mm
- net S$174: track 297.8 -> 285.4 mm, vias 0 -> 1
- net S$116: track 297.8 -> 285.4 mm, vias 0 -> 1
- net S$87: track 297.8 -> 285.4 mm, vias 0 -> 1
- net S$58: track 297.8 -> 285.4 mm, vias 0 -> 1
- net S$25: track 297.8 -> 285.4 mm, vias 0 -> 1
- net S$145: track 297.8 -> 285.4 mm, vias 0 -> 1
- net S$86: track 156.0 -> 151.4 mm
- net S$115: track 156.0 -> 151.4 mm
- net S$144: track 156.0 -> 151.4 mm
- net S$57: track 156.0 -> 151.4 mm
- net S$173: track 156.0 -> 151.4 mm

Commit message: pcb update
Parts:
- E$102: device capacitor-wima:C2.5-2 -> transistor:TO92-CBE
- E$104: device transistor:TO92-CBE -> capacitor-wima:C5B7.2
- E$206, E$310, E$414, E$518, E$622: device capacitor-wima:C2.5-2 -> diode:ZDIO-10
- E$207, E$311, E$415, E$519, E$623: device diode:ZDIO-10 -> switch:255SB
- E$208, E$312, E$416, E$520, E$624: device switch:255SB -> capacitor-wima:C5B7.2
- moved E$104 111.8 mm to (27.9, 94.0), turned to 90 degrees
- moved E$102 109.7 mm to (137.2, 92.7), turned to 270 degrees
- moved E$623 72.8 mm to (121.9, -58.4), turned to 0 degrees
- moved E$415 71.0 mm to (121.9, 12.7), turned to 0 degrees
- moved E$519 70.6 mm to (27.9, -58.4), turned to 0 degrees
- moved E$207 69.4 mm to (121.9, 83.8), turned to 0 degrees
- moved E$311 68.7 mm to (27.9, 12.7), turned to 0 degrees
- moved E$310 65.1 mm to (88.9, -15.2)
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Connections:
- removed net S$100: E$338.A, E$339.C
- removed net S$101: E$337.A, E$340.C
- removed net S$111: E$315.B, E$325.2
- removed net S$125: E$433.B, E$435.C, E$446.1
- removed net S$126: E$433.E
- removed net S$131: E$445.1, E$480.1
- removed net S$132: E$432.1, E$478.1
- removed net S$142: E$434.B, E$448.2
- removed net S$156: E$540.E
- removed net S$157: E$538.C, E$540.B, E$551.1
- removed net S$162: E$533.1, E$583.1
- removed net S$173: E$521.C, E$524.C, E$529.C, E$530.C, E$534.2, E$535.2, E$558.1, E$573.1, E$574.1, E$620.2, E$622.2, E$624.1
- removed net S$32: E$104.E
- removed net S$38: E$121.B, E$123.C, E$134.1
- removed net S$39: E$121.E
- removed net S$49: E$114.A, E$115.C
- removed net S$63: E$212.E
- removed net S$64: E$210.C, E$212.B, E$223.1
- removed net S$69: E$228.E
- removed net S$70: E$226.C, E$228.B, E$239.1
- removed net S$80: E$225.C, E$228.C, E$233.C, E$234.C, E$238.2, E$239.2, E$276.1, E$311.C
- new net S$105: E$330.C, E$332.B, E$343.1
- new net S$117: E$315.B, E$325.2
- new net S$118: E$314.B, E$328.2
- new net S$123: E$313.C, E$316.C, E$321.C, E$322.C, E$326.2, E$327.2, E$350.1, E$365.1, E$366.1, E$412.2, E$415.3, E$416.2
- new net S$124: E$415.1
- new net S$134: E$433.E
- new net S$146: E$433.C, E$436.C, E$441.C, E$442.C, E$446.2, E$447.2, E$484.1, E$518.C
- new net S$147: E$448.1, E$481.1
- new net S$152: E$418.E, E$419.E, E$427.A, E$428.A, E$434.E, E$435.E, E$443.A, E$444.A, E$485.1, E$511.1, E$516.1, E$520.1
- new net S$153: E$519.2
- new net S$175: E$530.A, E$531.C
- new net S$176: E$529.A, E$532.C
- new net S$177: E$537.C, E$540.C, E$545.C, E$546.C, E$550.2, E$551.2, E$588.1, E$622.C
- new net S$178: E$552.1, E$585.1
- new net S$179: E$523.B, E$533.2
- new net S$180: E$522.B, E$536.2
- new net S$181: E$538.B, E$552.2
- new net S$182: E$539.B, E$549.2
- new net S$183: E$522.E, E$523.E, E$531.A, E$532.A, E$538.E, E$539.E, E$547.A, E$548.A, E$589.1, E$615.1, E$620.1, E$624.1
- new net S$184: E$623.2
- new net S$185: E$521.C, E$524.C, E$529.C, E$530.C, E$534.2, E$535.2, E$558.1, E$573.1, E$574.1, E$620.2, E$623.3, E$624.2
- new net S$186: E$623.1
- new net S$29: E$101.1, E$104.1, E$18.A, E$19.A, E$2.E, E$3.E, E$46.A, E$47.A, E$6.E, E$7.E, E$71.1, E$97.1
- new net S$35: E$108.E
- new net S$37: E$106.C, E$108.B, E$119.1
- new net S$47: E$120.1, E$166.1
- new net S$59: E$106.E, E$107.E, E$115.A, E$116.A, E$122.E, E$123.E, E$131.A, E$132.A, E$173.1, E$199.1, E$204.1, E$208.1
- new net S$60: E$207.2
- new net S$65: E$209.B, E$211.C, E$222.1
- new net S$66: E$209.E
- new net S$76: E$233.A, E$236.C
- new net S$88: E$226.B, E$240.2
- new net S$89: E$227.B, E$237.2
- net S$102: now also E$329.B, E$331.C, E$342.1; no longer E$341.1, E$376.1
- net S$103: now also E$329.E; no longer E$328.1, E$374.1
- net S$104: now also E$332.E; no longer E$325.1, E$375.1
- net S$106: now also E$338.A, E$339.C; no longer E$388.1
- net S$107: now also E$337.A, E$340.C; no longer E$322.A, E$323.C
- net S$108: now also E$341.1, E$376.1; no longer E$321.A, E$324.C
- net S$109: now also E$328.1, E$374.1; no longer E$329.C, E$332.C, E$337.C, E$338.C, E$342.2, E$343.2, E$380.1, E$415.C
- net S$110: now also E$325.1, E$375.1; no longer E$344.1, E$377.1
- net S$112: now also E$388.1; no longer E$314.B, E$328.2
- net S$113: now also E$322.A, E$323.C; no longer E$330.B, E$344.2
- net S$114: now also E$321.A, E$324.C; no longer E$331.B, E$341.2
- net S$115: now also E$329.C, E$332.C, E$337.C, E$338.C, E$342.2, E$343.2, E$380.1, E$414.C; no longer E$313.C, E$316.C, E$321.C, E$322.C, E$326.2, E$327.2, E$350.1, E$365.1, E$366.1, E$412.2, E$414.2, E$416.1
- net S$116: now also E$344.1, E$377.1; no longer E$314.E, E$315.E, E$323.A, E$324.A, E$330.E, E$331.E, E$339.A, E$340.A, E$381.1, E$407.1, E$412.1, E$414.1
- net S$119: now also E$330.B, E$344.2; no longer E$417.B, E$419.C, E$430.1
- net S$120: now also E$331.B, E$341.2; no longer E$417.E
- net S$121: now also E$314.E, E$315.E, E$323.A, E$324.A, E$330.E, E$331.E, E$339.A, E$340.A, E$381.1, E$407.1, E$412.1, E$416.1; no longer E$420.E
- net S$122: now also E$415.2; no longer E$418.C, E$420.B, E$431.1
- net S$127: now also E$417.B, E$419.C, E$430.1; no longer E$436.E
- net S$128: now also E$417.E; no longer E$434.C, E$436.B, E$447.1
- net S$129: now also E$420.E; no longer E$442.A, E$443.C
- net S$130: now also E$418.C, E$420.B, E$431.1; no longer E$441.A, E$444.C
- net S$133: now also E$433.B, E$435.C, E$446.1; no longer E$429.1, E$479.1
- net S$135: now also E$436.E; no longer E$492.1
- net S$136: now also E$434.C, E$436.B, E$447.1; no longer E$426.A, E$427.C
- net S$137: now also E$442.A, E$443.C; no longer E$425.A, E$428.C
- net S$138: now also E$441.A, E$444.C; no longer E$433.C, E$436.C, E$441.C, E$442.C, E$446.2, E$447.2, E$484.1, E$519.C
- net S$139: now also E$445.1, E$480.1; no longer E$448.1, E$481.1
- net S$140: now also E$432.1, E$478.1; no longer E$419.B, E$429.2
- net S$141: now also E$429.1, E$479.1; no longer E$418.B, E$432.2
- net S$143: now also E$492.1; no longer E$435.B, E$445.2
- net S$144: now also E$426.A, E$427.C; no longer E$417.C, E$420.C, E$425.C, E$426.C, E$430.2, E$431.2, E$454.1, E$469.1, E$470.1, E$516.2, E$518.2, E$520.1
- net S$145: now also E$425.A, E$428.C; no longer E$418.E, E$419.E, E$427.A, E$428.A, E$434.E, E$435.E, E$443.A, E$444.A, E$485.1, E$511.1, E$516.1, E$518.1
- net S$148: now also E$419.B, E$429.2; no longer E$521.B, E$523.C, E$534.1
- net S$149: now also E$418.B, E$432.2; no longer E$521.E
- net S$150: now also E$434.B, E$448.2; no longer E$524.E
- net S$151: now also E$435.B, E$445.2; no longer E$522.C, E$524.B, E$535.1
- net S$154: now also E$417.C, E$420.C, E$425.C, E$426.C, E$430.2, E$431.2, E$454.1, E$469.1, E$470.1, E$516.2, E$519.3, E$520.2; no longer E$537.B, E$539.C, E$550.1
- net S$155: now also E$519.1; no longer E$537.E
- net S$158: now also E$521.B, E$523.C, E$534.1; no longer E$546.A, E$547.C
- net S$159: now also E$521.E; no longer E$545.A, E$548.C
- net S$160: now also E$524.E; no longer E$549.1, E$584.1
- net S$161: now also E$522.C, E$524.B, E$535.1; no longer E$536.1, E$582.1
- net S$164: now also E$537.B, E$539.C, E$550.1; no longer E$596.1
- net S$165: now also E$537.E; no longer E$530.A, E$531.C
- net S$166: now also E$540.E; no longer E$529.A, E$532.C
- net S$167: now also E$538.C, E$540.B, E$551.1; no longer E$537.C, E$540.C, E$545.C, E$546.C, E$550.2, E$551.2, E$588.1, E$623.C
- net S$168: now also E$546.A, E$547.C; no longer E$552.1, E$585.1
- net S$169: now also E$545.A, E$548.C; no longer E$523.B, E$533.2
- net S$170: now also E$549.1, E$584.1; no longer E$522.B, E$536.2
- net S$171: now also E$536.1, E$582.1; no longer E$538.B, E$552.2
- net S$172: now also E$533.1, E$583.1; no longer E$539.B, E$549.2
- net S$174: now also E$596.1; no longer E$522.E, E$523.E, E$531.A, E$532.A, E$538.E, E$539.E, E$547.A, E$548.A, E$589.1, E$615.1, E$620.1, E$622.1
- net S$20: no longer E$1.C, E$101.2, E$102.2, E$29.1, E$4.C, E$44.C, E$45.C, E$49.2, E$50.2, E$58.1, E$59.1
- net S$25: now also E$1.C, E$101.2, E$103.3, E$104.2, E$29.1, E$4.C, E$44.C, E$45.C, E$49.2, E$50.2, E$58.1, E$59.1; no longer E$101.1, E$102.1, E$18.A, E$19.A, E$2.E, E$3.E, E$46.A, E$47.A, E$6.E, E$7.E, E$71.1, E$97.1
- net S$31: now also E$103.2; no longer E$104.B, E$107.C, E$118.1
- net S$33: now also E$102.B, E$107.C, E$118.1; no longer E$108.E
- net S$34: now also E$102.E; no longer E$106.C, E$108.B, E$119.1
- net S$40: now also E$121.B, E$123.C, E$134.1; no longer E$124.E
- net S$41: now also E$121.E; no longer E$122.C, E$124.B, E$135.1
- net S$42: now also E$124.E; no longer E$130.A, E$131.C
- net S$43: now also E$122.C, E$124.B, E$135.1; no longer E$129.A, E$132.C
- net S$44: now also E$130.A, E$131.C; no longer E$133.1, E$168.1
- net S$45: now also E$129.A, E$132.C; no longer E$120.1, E$166.1
- net S$46: now also E$133.1, E$168.1; no longer E$117.1, E$167.1
- net S$48: now also E$117.1, E$167.1; no longer E$180.1
- net S$50: now also E$180.1; no longer E$113.A, E$116.C
- net S$51: now also E$114.A, E$115.C; no longer E$121.C, E$124.C, E$129.C, E$130.C, E$134.2, E$135.2, E$172.1, E$207.C
- net S$52: now also E$113.A, E$116.C; no longer E$136.1, E$169.1
- net S$53: now also E$121.C, E$124.C, E$129.C, E$130.C, E$134.2, E$135.2, E$172.1, E$206.C; no longer E$107.B, E$117.2
- net S$54: now also E$136.1, E$169.1; no longer E$106.B, E$120.2
- net S$55: now also E$107.B, E$117.2; no longer E$122.B, E$136.2
- net S$56: now also E$106.B, E$120.2; no longer E$123.B, E$133.2
- net S$57: now also E$122.B, E$136.2; no longer E$104.C, E$108.C, E$113.C, E$114.C, E$118.2, E$119.2, E$142.1, E$157.1, E$158.1, E$204.2, E$206.2, E$208.1
- net S$58: now also E$123.B, E$133.2; no longer E$106.E, E$107.E, E$115.A, E$116.A, E$122.E, E$123.E, E$131.A, E$132.A, E$173.1, E$199.1, E$204.1, E$206.1
- net S$61: now also E$102.C, E$108.C, E$113.C, E$114.C, E$118.2, E$119.2, E$142.1, E$157.1, E$158.1, E$204.2, E$207.3, E$208.2; no longer E$209.B, E$211.C, E$222.1
- net S$62: now also E$207.1; no longer E$209.E
- net S$67: now also E$212.E; no longer E$225.B, E$227.C, E$238.1
- net S$68: now also E$210.C, E$212.B, E$223.1; no longer E$225.E
- net S$71: now also E$225.B, E$227.C, E$238.1; no longer E$234.A, E$235.C
- net S$72: now also E$225.E; no longer E$233.A, E$236.C
- net S$73: now also E$228.E; no longer E$237.1, E$272.1
- net S$74: now also E$226.C, E$228.B, E$239.1; no longer E$224.1, E$270.1
- net S$75: now also E$234.A, E$235.C; no longer E$221.1, E$271.1
- net S$77: now also E$237.1, E$272.1; no longer E$284.1
- net S$78: now also E$224.1, E$270.1; no longer E$218.A, E$219.C
- net S$79: now also E$221.1, E$271.1; no longer E$217.A, E$220.C
- net S$81: now also E$284.1; no longer E$240.1, E$273.1
- net S$82: now also E$218.A, E$219.C; no longer E$211.B, E$221.2
- net S$83: now also E$217.A, E$220.C; no longer E$210.B, E$224.2
- net S$84: now also E$225.C, E$228.C, E$233.C, E$234.C, E$238.2, E$239.2, E$276.1, E$310.C; no longer E$226.B, E$240.2
- net S$85: now also E$240.1, E$273.1; no longer E$227.B, E$237.2
- net S$86: now also E$211.B, E$221.2; no longer E$209.C, E$212.C, E$217.C, E$218.C, E$222.2, E$223.2, E$246.1, E$261.1, E$262.1, E$308.2, E$310.2, E$312.1
- net S$87: now also E$210.B, E$224.2; no longer E$210.E, E$211.E, E$219.A, E$220.A, E$226.E, E$227.E, E$235.A, E$236.A, E$277.1, E$303.1, E$308.1, E$310.1
- net S$90: now also E$210.E, E$211.E, E$219.A, E$220.A, E$226.E, E$227.E, E$235.A, E$236.A, E$277.1, E$303.1, E$308.1, E$312.1; no longer E$313.B, E$315.C, E$326.1
- net S$91: now also E$311.2; no longer E$313.E
- net S$92: now also E$209.C, E$212.C, E$217.C, E$218.C, E$222.2, E$223.2, E$246.1, E$261.1, E$262.1, E$308.2, E$311.3, E$312.2; no longer E$316.E
- net S$93: now also E$311.1; no longer E$314.C, E$316.B, E$327.1
- net S$96: now also E$313.B, E$315.C, E$326.1; no longer E$329.B, E$331.C, E$342.1
- net S$97: now also E$313.E; no longer E$329.E
- net S$98: now also E$316.E; no longer E$332.E
- net S$99: now also E$314.C, E$316.B, E$327.1; no longer E$330.C, E$332.B, E$343.1
Routing:
- net S$183: track 0.00 -> 301.2 mm, vias 0 -> 1
- net S$121: track 8.67 -> 301.2 mm, vias 0 -> 1
- net S$90: track 18.8 -> 301.2 mm, vias 0 -> 1
- net S$152: track 19.6 -> 301.2 mm, vias 0 -> 1
- net S$59: track 19.6 -> 301.2 mm, vias 0 -> 1
- net S$29: track 19.6 -> 301.2 mm, vias 0 -> 1
- net S$87: track 285.4 -> 4.34 mm, vias 1 -> 0
- net S$58: track 285.4 -> 4.34 mm, vias 1 -> 0
- net S$145: track 285.4 -> 5.08 mm, vias 1 -> 2
- net S$116: track 285.4 -> 5.08 mm, vias 1 -> 0
- net S$174: track 285.4 -> 39.5 mm, vias 1 -> 0
- net S$185: track 0.00 -> 161.3 mm
- net S$92: track 8.67 -> 161.3 mm
- net S$173: track 151.4 -> 0.00 mm
- net S$57: track 151.4 -> 4.34 mm
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- added copper zone on layer 16, net S$111
- added copper zone on layer 16, net S$142
- added copper zone on layer 16, net S$173
- added copper zone on layer 16, net S$49
- added copper zone on layer 16, net S$80
- removed copper zone on layer 16, net S$105
- removed copper zone on layer 16, net S$134
- removed copper zone on layer 16, net S$163
- removed copper zone on layer 16, net S$47
- removed copper zone on layer 16, net S$76
