File: microcap/pcb/testK.brd (EAGLE design)
At the start: 103 parts

Commit message: pcb test update
Changed lines of the file:
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@@
 <signal name="S$24">
 <polygon width="0.4064" layer="16">
-<vertex x="113.03" y="31.75"/>
-<vertex x="29.21" y="31.75"/>
-<vertex x="29.21" y="100.33"/>
-<vertex x="113.03" y="100.33"/>
+<vertex x="114.3" y="30.48"/>
+<vertex x="27.94" y="30.48"/>
+<vertex x="27.94" y="101.6"/>
+<vertex x="114.3" y="101.6"/>
 </polygon>
 </signal>

Commit message: pcb update
Parts:
- moved E$20 1.27 mm to (34.3, 52.1)
- moved E$23 1.27 mm to (78.7, 52.1)
- moved E$48 1.27 mm to (34.3, 74.9)
- moved E$51 1.27 mm to (78.7, 74.9)
Routing:
- net S$23: track 54.0 -> 52.7 mm
- net S$18: track 9.94 -> 8.67 mm
- net S$36: track 61.6 -> 60.3 mm
- net S$28: track 90.6 -> 89.8 mm
- net S$17: track 3.81 -> 4.34 mm
- net S$21: track 3.81 -> 4.34 mm
- net S$6: track 3.81 -> 4.34 mm
- net S$5: track 3.81 -> 4.34 mm
- net S$15: track 5.61 -> 5.08 mm
Changed lines of the file:
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@@
 <element name="E$46" library="diode" package="C2992" value="" x="54.61" y="77.47" rot="R270"/>
 <element name="E$47" library="diode" package="C2992" value="" x="58.42" y="77.47" rot="R270"/>
-<element name="E$48" library="resistor" package="0207/10" value="" x="34.29" y="76.2" rot="R90"/>
+<element name="E$48" library="resistor" package="0207/10" value="" x="34.29" y="74.93" rot="R90"/>
 <element name="E$49" library="resistor" package="0207/10" value="" x="38.1" y="91.44" rot="R90"/>
 <element name="E$50" library="resistor" package="0207/10" value="" x="74.93" y="91.44" rot="R90"/>
-<element name="E$51" library="resistor" package="0207/10" value="" x="78.74" y="76.2" rot="R90"/>
+<element name="E$51" library="resistor" package="0207/10" value="" x="78.74" y="74.93" rot="R90"/>
 <element name="E$5" library="transistor" package="TO92-CBE" value="" x="43.18" y="57.15" rot="R270"/>
 <element name="E$6" library="transistor" package="TO92-CBE" value="" x="74.93" y="45.72" rot="R270"/>
@@
 <element name="E$18" library="diode" package="C2992" value="" x="54.61" y="41.91" rot="R270"/>
 <element name="E$19" library="diode" package="C2992" value="" x="58.42" y="41.91" rot="R270"/>
-<element name="E$20" library="resistor" package="0207/10" value="" x="34.29" y="50.8" rot="R270"/>
+<element name="E$20" library="resistor" package="0207/10" value="" x="34.29" y="52.07" rot="R270"/>
 <element name="E$21" library="resistor" package="0207/10" value="" x="38.1" y="55.88" rot="R90"/>
 <element name="E$22" library="resistor" package="0207/10" value="" x="74.93" y="55.88" rot="R90"/>
-<element name="E$23" library="resistor" package="0207/10" value="" x="78.74" y="50.8" rot="R270"/>
+<element name="E$23" library="resistor" package="0207/10" value="" x="78.74" y="52.07" rot="R270"/>
 <element name="E$24" library="pinhead" package="1X01" value="" x="83.82" y="87.63"/>
 <element name="E$25" library="pinhead" package="1X01" value="" x="83.82" y="85.09"/>
@@
 <wire x1="74.93" y1="83.82" x2="68.58" y2="83.82" width="0.4064" layer="16"/>
 </signal>
-<signal name="S$5">
-<contactref element="E$3" pad="B"/>
-<contactref element="E$48" pad="2"/>
-<wire x1="38.1" y1="81.28" x2="34.29" y2="81.28" width="0.4064" layer="16"/>
-</signal>
-<signal name="S$6">
-<contactref element="E$2" pad="B"/>
-<contactref element="E$51" pad="2"/>
-<wire x1="74.93" y1="81.28" x2="78.74" y2="81.28" width="0.4064" layer="16"/>
-</signal>
 <signal name="S$1">
 <wire x1="49.53" y1="54.61" x2="49.53" y2="49.53" width="0.4064" layer="16"/>
@@
 <wire x1="74.93" y1="48.26" x2="68.58" y2="48.26" width="0.4064" layer="16"/>
 </signal>
-<signal name="S$17">
-<contactref element="E$6" pad="B"/>
-<contactref element="E$23" pad="2"/>
-<wire x1="74.93" y1="45.72" x2="78.74" y2="45.72" width="0.4064" layer="16"/>
-</signal>
-<signal name="S$21">
-<contactref element="E$7" pad="B"/>
-<contactref element="E$20" pad="2"/>
-<wire x1="38.1" y1="45.72" x2="34.29" y2="45.72" width="0.4064" layer="16"/>
-</signal>
 <signal name="S$12">
 <contactref element="E$18" pad="C"/>
@@
 <wire x1="74.93" y1="66.04" x2="35.56" y2="66.04" width="0.4064" layer="16"/>
 <contactref element="E$20" pad="1"/>
-<wire x1="34.29" y1="55.88" x2="34.29" y2="64.77" width="0.4064" layer="16"/>
+<wire x1="34.29" y1="57.15" x2="34.29" y2="64.77" width="0.4064" layer="16"/>
 <wire x1="34.29" y1="64.77" x2="35.56" y2="66.04" width="0.4064" layer="16"/>
 <contactref element="E$66" pad="1"/>
@@
 <wire x1="81.28" y1="64.77" x2="83.82" y2="64.77" width="0.4064" layer="16"/>
 <contactref element="E$51" pad="1"/>
-<wire x1="78.74" y1="71.12" x2="78.74" y2="67.31" width="0.4064" layer="16"/>
+<wire x1="78.74" y1="69.85" x2="78.74" y2="67.31" width="0.4064" layer="16"/>
 <wire x1="81.28" y1="64.77" x2="78.74" y2="67.31" width="0.4064" layer="16"/>
 </signal>
@@
 <contactref element="E$48" pad="1"/>
 <wire x1="74.93" y1="68.58" x2="35.56" y2="68.58" width="0.4064" layer="16"/>
-<wire x1="34.29" y1="71.12" x2="34.29" y2="69.85" width="0.4064" layer="16"/>
 <wire x1="34.29" y1="69.85" x2="35.56" y2="68.58" width="0.4064" layer="16"/>
 <contactref element="E$65" pad="1"/>
@@
 <contactref element="E$102" pad="1"/>
 <wire x1="33.02" y1="95.25" x2="30.48" y2="92.71" width="0.4064" layer="16"/>
-<wire x1="38.1" y1="78.74" x2="38.1" y2="76.2" width="0.4064" layer="16"/>
-<wire x1="38.1" y1="76.2" x2="38.1" y2="72.39" width="0.4064" layer="16"/>
-<wire x1="38.1" y1="76.2" x2="30.48" y2="76.2" width="0.4064" layer="16"/>
-<wire x1="30.48" y1="92.71" x2="30.48" y2="76.2" width="0.4064" layer="16"/>
-<wire x1="30.48" y1="76.2" x2="30.48" y2="38.1" width="0.4064" layer="16"/>
+<wire x1="38.1" y1="78.74" x2="38.1" y2="74.93" width="0.4064" layer="16"/>
+<wire x1="38.1" y1="74.93" x2="38.1" y2="72.39" width="0.4064" layer="16"/>
+<wire x1="38.1" y1="74.93" x2="30.48" y2="74.93" width="0.4064" layer="16"/>
+<wire x1="30.48" y1="92.71" x2="30.48" y2="74.93" width="0.4064" layer="16"/>
+<wire x1="30.48" y1="74.93" x2="30.48" y2="38.1" width="0.4064" layer="16"/>
 <wire x1="30.48" y1="38.1" x2="33.02" y2="35.56" width="0.4064" layer="16"/>
 <wire x1="69.85" y1="45.72" x2="68.58" y2="45.72" width="0.4064" layer="16"/>
@@
 <wire x1="69.85" y1="63.5" x2="73.66" y2="63.5" width="0.4064" layer="16"/>
 <wire x1="73.66" y1="63.5" x2="74.93" y2="62.23" width="0.4064" layer="16"/>
-<wire x1="78.74" y1="52.07" x2="78.74" y2="50.8" width="0.4064" layer="16"/>
-<wire x1="74.93" y1="55.88" x2="78.74" y2="52.07" width="0.4064" layer="16"/>
+<wire x1="74.93" y1="55.88" x2="81.28" y2="49.53" width="0.4064" layer="16"/>
 <contactref element="E$22" pad="2"/>
 <wire x1="74.93" y1="60.96" x2="74.93" y2="55.88" width="0.4064" layer="16"/>
@@
 <contactref element="E$105" pad="C"/>
 <wire x1="88.9" y1="49.53" x2="88.9" y2="50.8" width="0.4064" layer="16"/>
-<wire x1="80.01" y1="49.53" x2="83.82" y2="49.53" width="0.4064" layer="16"/>
-<wire x1="80.01" y1="49.53" x2="78.74" y2="50.8" width="0.4064" layer="16"/>
+<wire x1="81.28" y1="49.53" x2="83.82" y2="49.53" width="0.4064" layer="16"/>
 </signal>
 <signal name="S$15">
 <contactref element="E$67" pad="1"/>
-<wire x1="83.82" y1="57.15" x2="80.01" y2="57.15" width="0.4064" layer="16"/>
+<wire x1="83.82" y1="57.15" x2="78.74" y2="57.15" width="0.4064" layer="16"/>
 <contactref element="E$23" pad="1"/>
-<wire x1="80.01" y1="57.15" x2="78.74" y2="55.88" width="0.4064" layer="16"/>
+</signal>
+<signal name="S$5">
+<contactref element="E$48" pad="2"/>
+<wire x1="34.29" y1="80.01" x2="35.56" y2="81.28" width="0.4064" layer="16"/>
+<contactref element="E$3" pad="B"/>
+<wire x1="35.56" y1="81.28" x2="38.1" y2="81.28" width="0.4064" layer="16"/>
+</signal>
+<signal name="S$6">
+<contactref element="E$51" pad="2"/>
+<wire x1="78.74" y1="80.01" x2="77.47" y2="81.28" width="0.4064" layer="16"/>
+<contactref element="E$2" pad="B"/>
+<wire x1="77.47" y1="81.28" x2="74.93" y2="81.28" width="0.4064" layer="16"/>
+</signal>
+<signal name="S$17">
+<contactref element="E$23" pad="2"/>
+<wire x1="78.74" y1="46.99" x2="77.47" y2="45.72" width="0.4064" layer="16"/>
+<contactref element="E$6" pad="B"/>
+<wire x1="77.47" y1="45.72" x2="74.93" y2="45.72" width="0.4064" layer="16"/>
+</signal>
+<signal name="S$21">
+<contactref element="E$20" pad="2"/>
+<wire x1="34.29" y1="46.99" x2="35.56" y2="45.72" width="0.4064" layer="16"/>
+<contactref element="E$7" pad="B"/>
+<wire x1="35.56" y1="45.72" x2="38.1" y2="45.72" width="0.4064" layer="16"/>
 </signal>
 </signals>
