File: microcap/pcb/testL.brd (EAGLE design)
At the start: 104 parts

Commit message: pcb update
Connections:
- removed net S$29: E$1.C, E$101.2, E$102.2, E$103.2, E$29.1, E$4.C, E$44.C, E$45.C, E$49.2, E$50.2, E$58.1, E$59.1
- new net S$20: E$1.C, E$101.2, E$102.2, E$103.1, E$29.1, E$4.C, E$44.C, E$45.C, E$49.2, E$50.2, E$58.1, E$59.1
- net S$25: no longer E$103.1
Routing:
- net S$29: track 156.0 -> 0.00 mm
- net S$20: track 0.00 -> 151.4 mm
- net S$25: track 297.8 -> 285.4 mm, vias 0 -> 1
Changed lines of the file:
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@@
 <wire x1="35.56" y1="45.72" x2="38.1" y2="45.72" width="0.4064" layer="16"/>
 </signal>
-<signal name="S$29">
-<contactref element="E$58" pad="1"/>
-<contactref element="E$59" pad="1"/>
-<wire x1="86.36" y1="92.71" x2="83.82" y2="92.71" width="0.4064" layer="16"/>
+<signal name="S$20">
+<wire x1="93.98" y1="54.61" x2="93.98" y2="55.88" width="0.4064" layer="16"/>
+<wire x1="93.98" y1="55.88" x2="88.9" y2="60.96" width="0.4064" layer="16"/>
 <contactref element="E$101" pad="2"/>
-<contactref element="E$29" pad="1"/>
-<wire x1="86.36" y1="92.71" x2="88.9" y2="92.71" width="0.4064" layer="16"/>
-<wire x1="88.9" y1="87.63" x2="88.9" y2="92.71" width="0.4064" layer="16"/>
 <wire x1="95.25" y1="87.63" x2="88.9" y2="87.63" width="0.4064" layer="16"/>
 <wire x1="88.9" y1="60.96" x2="88.9" y2="87.63" width="0.4064" layer="16"/>
-<wire x1="93.98" y1="55.88" x2="88.9" y2="60.96" width="0.4064" layer="16"/>
-<wire x1="93.98" y1="54.61" x2="93.98" y2="55.88" width="0.4064" layer="16"/>
+<contactref element="E$29" pad="1"/>
+<wire x1="88.9" y1="87.63" x2="88.9" y2="92.71" width="0.4064" layer="16"/>
+<contactref element="E$59" pad="1"/>
+<wire x1="86.36" y1="92.71" x2="88.9" y2="92.71" width="0.4064" layer="16"/>
+<contactref element="E$58" pad="1"/>
+<wire x1="86.36" y1="92.71" x2="83.82" y2="92.71" width="0.4064" layer="16"/>
+<wire x1="83.82" y1="92.71" x2="78.74" y2="92.71" width="0.4064" layer="16"/>
+<contactref element="E$50" pad="2"/>
+<wire x1="78.74" y1="92.71" x2="74.93" y2="96.52" width="0.4064" layer="16"/>
+<wire x1="63.5" y1="92.71" x2="62.23" y2="92.71" width="0.4064" layer="16"/>
+<wire x1="72.39" y1="99.06" x2="74.93" y2="96.52" width="0.4064" layer="16"/>
 <contactref element="E$4" pad="C"/>
 <wire x1="69.85" y1="95.25" x2="69.85" y2="99.06" width="0.4064" layer="16"/>
+<wire x1="69.85" y1="99.06" x2="72.39" y2="99.06" width="0.4064" layer="16"/>
+<wire x1="62.23" y1="92.71" x2="60.96" y2="93.98" width="0.4064" layer="16"/>
+<contactref element="E$44" pad="C"/>
 <wire x1="60.96" y1="93.98" x2="60.96" y2="99.06" width="0.4064" layer="16"/>
-<wire x1="63.5" y1="92.71" x2="62.23" y2="92.71" width="0.4064" layer="16"/>
-<wire x1="62.23" y1="92.71" x2="60.96" y2="93.98" width="0.4064" layer="16"/>
-<contactref element="E$50" pad="2"/>
-<contactref element="E$44" pad="C"/>
+<wire x1="60.96" y1="99.06" x2="69.85" y2="99.06" width="0.4064" layer="16"/>
+<wire x1="49.53" y1="92.71" x2="50.8" y2="92.71" width="0.4064" layer="16"/>
 <contactref element="E$45" pad="C"/>
-<wire x1="49.53" y1="92.71" x2="50.8" y2="92.71" width="0.4064" layer="16"/>
+<wire x1="58.42" y1="99.06" x2="60.96" y2="99.06" width="0.4064" layer="16"/>
+<wire x1="58.42" y1="97.79" x2="58.42" y2="99.06" width="0.4064" layer="16"/>
+<wire x1="54.61" y1="99.06" x2="58.42" y2="99.06" width="0.4064" layer="16"/>
+<wire x1="54.61" y1="97.79" x2="54.61" y2="99.06" width="0.4064" layer="16"/>
 <wire x1="50.8" y1="92.71" x2="52.07" y2="93.98" width="0.4064" layer="16"/>
 <wire x1="52.07" y1="93.98" x2="52.07" y2="99.06" width="0.4064" layer="16"/>
-<wire x1="78.74" y1="92.71" x2="74.93" y2="96.52" width="0.4064" layer="16"/>
 <wire x1="52.07" y1="99.06" x2="54.61" y2="99.06" width="0.4064" layer="16"/>
-<wire x1="54.61" y1="99.06" x2="58.42" y2="99.06" width="0.4064" layer="16"/>
-<wire x1="58.42" y1="99.06" x2="60.96" y2="99.06" width="0.4064" layer="16"/>
-<wire x1="60.96" y1="99.06" x2="69.85" y2="99.06" width="0.4064" layer="16"/>
-<wire x1="69.85" y1="99.06" x2="72.39" y2="99.06" width="0.4064" layer="16"/>
-<wire x1="72.39" y1="99.06" x2="74.93" y2="96.52" width="0.4064" layer="16"/>
-<wire x1="54.61" y1="97.79" x2="54.61" y2="99.06" width="0.4064" layer="16"/>
-<wire x1="58.42" y1="97.79" x2="58.42" y2="99.06" width="0.4064" layer="16"/>
 <contactref element="E$1" pad="C"/>
 <contactref element="E$49" pad="2"/>
 <wire x1="43.18" y1="95.25" x2="43.18" y2="99.06" width="0.4064" layer="16"/>
+<wire x1="52.07" y1="99.06" x2="43.18" y2="99.06" width="0.4064" layer="16"/>
 <wire x1="38.1" y1="99.06" x2="43.18" y2="99.06" width="0.4064" layer="16"/>
 <wire x1="38.1" y1="96.52" x2="38.1" y2="99.06" width="0.4064" layer="16"/>
-<wire x1="52.07" y1="99.06" x2="43.18" y2="99.06" width="0.4064" layer="16"/>
-<wire x1="83.82" y1="92.71" x2="78.74" y2="92.71" width="0.4064" layer="16"/>
-<contactref element="E$103" pad="2"/>
-<wire x1="27.94" y1="93.98" x2="30.48" y2="93.98" width="0.4064" layer="16"/>
-<wire x1="27.94" y1="93.98" x2="25.4" y2="93.98" width="0.4064" layer="16"/>
+<wire x1="38.1" y1="99.06" x2="35.56" y2="99.06" width="0.4064" layer="16"/>
+<contactref element="E$103" pad="1"/>
 <contactref element="E$102" pad="2"/>
-<wire x1="24.13" y1="92.71" x2="24.13" y2="87.63" width="0.4064" layer="16"/>
-<wire x1="27.94" y1="83.82" x2="24.13" y2="87.63" width="0.4064" layer="16"/>
-<wire x1="24.13" y1="92.71" x2="25.4" y2="93.98" width="0.4064" layer="16"/>
-<wire x1="38.1" y1="99.06" x2="35.56" y2="99.06" width="0.4064" layer="16"/>
-<wire x1="35.56" y1="99.06" x2="30.48" y2="93.98" width="0.4064" layer="16"/>
+<wire x1="30.48" y1="90.17" x2="27.94" y2="90.17" width="0.4064" layer="16"/>
+<wire x1="27.94" y1="90.17" x2="27.94" y2="83.82" width="0.4064" layer="16"/>
+<wire x1="30.48" y1="90.17" x2="33.02" y2="92.71" width="0.4064" layer="16"/>
+<wire x1="35.56" y1="99.06" x2="33.02" y2="96.52" width="0.4064" layer="16"/>
+<wire x1="33.02" y1="96.52" x2="33.02" y2="92.71" width="0.4064" layer="16"/>
 </signal>
 <signal name="S$25">
@@
 <wire x1="38.1" y1="78.74" x2="38.1" y2="74.93" width="0.4064" layer="16"/>
 <wire x1="38.1" y1="74.93" x2="38.1" y2="72.39" width="0.4064" layer="16"/>
-<wire x1="38.1" y1="74.93" x2="31.75" y2="74.93" width="0.4064" layer="16"/>
-<wire x1="30.48" y1="73.66" x2="30.48" y2="38.1" width="0.4064" layer="16"/>
+<wire x1="38.1" y1="74.93" x2="30.48" y2="74.93" width="0.4064" layer="16"/>
+<wire x1="30.48" y1="74.93" x2="30.48" y2="38.1" width="0.4064" layer="16"/>
 <wire x1="30.48" y1="38.1" x2="33.02" y2="35.56" width="0.4064" layer="16"/>
 <wire x1="69.85" y1="45.72" x2="68.58" y2="45.72" width="0.4064" layer="16"/>
@@
 <wire x1="82.55" y1="46.99" x2="76.2" y2="40.64" width="0.4064" layer="16"/>
 <wire x1="63.5" y1="36.83" x2="62.23" y2="35.56" width="0.4064" layer="16"/>
-<wire x1="30.48" y1="73.66" x2="31.75" y2="74.93" width="0.4064" layer="16"/>
-<wire x1="31.75" y1="74.93" x2="31.75" y2="81.28" width="0.4064" layer="16"/>
-<contactref element="E$103" pad="1"/>
-<wire x1="31.75" y1="81.28" x2="31.75" y2="88.9" width="0.4064" layer="16"/>
 <contactref element="E$102" pad="1"/>
-<wire x1="30.48" y1="90.17" x2="27.94" y2="90.17" width="0.4064" layer="16"/>
-<wire x1="27.94" y1="81.28" x2="31.75" y2="81.28" width="0.4064" layer="16"/>
-<wire x1="30.48" y1="90.17" x2="31.75" y2="88.9" width="0.4064" layer="16"/>
+<wire x1="27.94" y1="81.28" x2="27.94" y2="74.93" width="0.4064" layer="16"/>
+<via x="27.94" y="74.93" extent="1-16" drill="0.6" shape="octagon"/>
+<wire x1="27.94" y1="74.93" x2="30.48" y2="74.93" width="0.4064" layer="16"/>
 </signal>
 </signals>
