File: microcap/pcb/testM.brd (EAGLE design)
At the start: 104 parts

Commit message: pcb update
Parts:
- moved E$103 15.2 mm to (26.7, 78.7)
- moved E$104 12.8 mm to (27.9, 94.0)
Connections:
- net S$25 renamed S$29
- net S$20: now also E$104.2
Routing:
- net S$20: track 152.7 -> 168.4 mm
- net S$29: track 284.6 -> 297.8 mm
