File: microcap/pcb/testN.brd (EAGLE design)
At the start: 104 parts

Commit message: pcb update
Parts:
- moved E$104 12.8 mm to (27.9, 94.0)
- moved E$103 10.2 mm to (27.9, 83.8), turned to 0 degrees
Connections:
- new net S$29: E$101.1, E$104.1, E$18.A, E$19.A, E$2.E, E$3.E, E$46.A, E$47.A, E$6.E, E$7.E, E$71.1, E$97.1
- new net S$31: E$103.2
- net S$20: no longer E$1.C, E$101.2, E$29.1, E$4.C, E$44.C, E$45.C, E$49.2, E$50.2, E$58.1, E$59.1
- net S$25: now also E$1.C, E$101.2, E$103.3, E$104.2, E$29.1, E$4.C, E$44.C, E$45.C, E$49.2, E$50.2, E$58.1, E$59.1; no longer E$101.1, E$104.1, E$18.A, E$19.A, E$2.E, E$3.E, E$46.A, E$47.A, E$6.E, E$7.E, E$71.1, E$97.1
Routing:
- net S$29: track 0.00 -> 301.2 mm, vias 0 -> 1
- net S$20: track 152.7 -> 22.6 mm, vias 0 -> 1
- net S$25: track 284.6 -> 161.3 mm, vias 1 -> 0
- net S$31: track 0.00 -> 12.7 mm, vias 0 -> 1

Commit message: cleaning
Parts:
- turned E$105 to 270 degrees
Connections:
- removed net S$25: E$1.C, E$101.2, E$103.3, E$104.2, E$29.1, E$4.C, E$44.C, E$45.C, E$49.2, E$50.2, E$58.1, E$59.1
- new net S$30: E$1.C, E$101.2, E$103.3, E$104.2, E$105.C, E$29.1, E$4.C, E$44.C, E$45.C, E$49.2, E$50.2, E$58.1, E$59.1
- net S$28: now also E$105.A; no longer E$105.C
Routing:
- net S$30: track 0.00 -> 161.3 mm
- net S$25: track 161.3 -> 0.00 mm
Changed lines of the file:
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@@
 <layer number="19" name="Unrouted" color="6" fill="1" visible="yes" active="yes"/>
 <layer number="20" name="Dimension" color="15" fill="1" visible="yes" active="yes"/>
-<layer number="21" name="tPlace" color="7" fill="1" visible="no" active="yes"/>
-<layer number="22" name="bPlace" color="7" fill="1" visible="no" active="yes"/>
+<layer number="21" name="tPlace" color="7" fill="1" visible="yes" active="yes"/>
+<layer number="22" name="bPlace" color="7" fill="1" visible="yes" active="yes"/>
 <layer number="23" name="tOrigins" color="15" fill="1" visible="no" active="yes"/>
 <layer number="24" name="bOrigins" color="15" fill="1" visible="no" active="yes"/>
@@
 <element name="E$101" library="capacitor-wima" package="C5B2.5" value="" x="97.79" y="87.63" rot="R180"/>
 <element name="E$94" library="resistor" package="0207/10" value="" x="93.98" y="49.53" rot="R270.2"/>
-<element name="E$105" library="diode" package="ZDIO-10" value="" x="88.9" y="55.88" rot="R90"/>
+<element name="E$105" library="diode" package="ZDIO-10" value="" x="88.9" y="55.88" rot="R270"/>
 <element name="E$103" library="switch" package="255SB" value="" x="27.94" y="83.82"/>
 <element name="E$104" library="capacitor-wima" package="C5B7.2" value="" x="27.94" y="93.98" rot="R90"/>
@@
 <wire x1="58.42" y1="62.23" x2="58.42" y2="63.5" width="0.4064" layer="16"/>
 <contactref element="E$70" pad="1"/>
+<wire x1="81.28" y1="49.53" x2="83.82" y2="49.53" width="0.4064" layer="16"/>
 <wire x1="83.82" y1="49.53" x2="88.9" y2="49.53" width="0.4064" layer="16"/>
-<contactref element="E$105" pad="C"/>
+<contactref element="E$105" pad="A"/>
 <wire x1="88.9" y1="49.53" x2="88.9" y2="50.8" width="0.4064" layer="16"/>
-<wire x1="81.28" y1="49.53" x2="83.82" y2="49.53" width="0.4064" layer="16"/>
 </signal>
 <signal name="S$15">
@@
 <via x="27.94" y="71.12" extent="1-16" drill="0.6" shape="octagon"/>
 </signal>
-<signal name="S$25">
+<signal name="S$30">
+<wire x1="93.98" y1="54.61" x2="93.98" y2="55.88" width="0.4064" layer="16"/>
 <contactref element="E$103" pad="3"/>
 <wire x1="31.75" y1="83.82" x2="31.75" y2="85.09" width="0.4064" layer="16"/>
 <wire x1="31.75" y1="85.09" x2="29.21" y2="87.63" width="0.4064" layer="16"/>
-<wire x1="93.98" y1="54.61" x2="93.98" y2="55.88" width="0.4064" layer="16"/>
-<wire x1="93.98" y1="55.88" x2="88.9" y2="60.96" width="0.4064" layer="16"/>
 <contactref element="E$101" pad="2"/>
 <wire x1="95.25" y1="87.63" x2="88.9" y2="87.63" width="0.4064" layer="16"/>
-<wire x1="88.9" y1="60.96" x2="88.9" y2="87.63" width="0.4064" layer="16"/>
 <contactref element="E$29" pad="1"/>
+<contactref element="E$59" pad="1"/>
 <wire x1="88.9" y1="87.63" x2="88.9" y2="92.71" width="0.4064" layer="16"/>
-<contactref element="E$59" pad="1"/>
 <wire x1="86.36" y1="92.71" x2="88.9" y2="92.71" width="0.4064" layer="16"/>
 <contactref element="E$58" pad="1"/>
@@
 <wire x1="29.21" y1="87.63" x2="25.4" y2="87.63" width="0.4064" layer="16"/>
 <wire x1="25.4" y1="87.63" x2="24.13" y2="88.9" width="0.4064" layer="16"/>
+<contactref element="E$105" pad="C"/>
+<wire x1="88.9" y1="60.96" x2="88.9" y2="87.63" width="0.4064" layer="16"/>
+<wire x1="93.98" y1="55.88" x2="88.9" y2="60.96" width="0.4064" layer="16"/>
 </signal>
 <signal name="S$20">
