File: microcap/pcb/pcb_v4.brd (EAGLE design)
At the start: 104 parts

Commit message: pcb update
Connections:
- removed net S$31: E$103.2
- net S$28: now also E$103.2; no longer E$103.3
Routing:
- net S$31: track 12.7 -> 0.00 mm, vias 1 -> 0
- net S$28: track 262.1 -> 271.7 mm, vias 0 -> 1
Changed lines of the file:
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@@
 <wire x1="81.28" y1="49.53" x2="83.82" y2="49.53" width="0.4064" layer="16"/>
 <wire x1="83.82" y1="49.53" x2="87.63" y2="49.53" width="0.4064" layer="16"/>
-<contactref element="E$103" pad="3"/>
-<wire x1="31.75" y1="83.82" x2="31.75" y2="85.09" width="0.4064" layer="16"/>
-<wire x1="31.75" y1="85.09" x2="29.21" y2="87.63" width="0.4064" layer="16"/>
 <contactref element="E$101" pad="2"/>
 <wire x1="95.25" y1="87.63" x2="88.9" y2="87.63" width="0.4064" layer="16"/>
@@
 <wire x1="25.4" y1="96.52" x2="24.13" y2="95.25" width="0.4064" layer="16"/>
 <wire x1="24.13" y1="88.9" x2="24.13" y2="95.25" width="0.4064" layer="16"/>
-<wire x1="29.21" y1="87.63" x2="25.4" y2="87.63" width="0.4064" layer="16"/>
+<wire x1="26.67" y1="87.63" x2="25.4" y2="87.63" width="0.4064" layer="16"/>
 <wire x1="25.4" y1="87.63" x2="24.13" y2="88.9" width="0.4064" layer="16"/>
 <wire x1="88.9" y1="50.8" x2="88.9" y2="60.96" width="0.4064" layer="16"/>
@@
 <wire x1="88.9" y1="60.96" x2="91.44" y2="60.96" width="0.4064" layer="16"/>
 <wire x1="91.44" y1="60.96" x2="93.98" y2="58.42" width="0.4064" layer="16"/>
-<wire x1="93.98" y1="54.61" x2="93.98" y2="55.88" width="0.4064" layer="16"/>
-<wire x1="93.98" y1="58.42" x2="93.98" y2="55.88" width="0.4064" layer="16"/>
+<wire x1="93.98" y1="58.42" x2="93.98" y2="54.61" width="0.4064" layer="16"/>
+<contactref element="E$103" pad="2"/>
+<wire x1="27.94" y1="83.82" x2="27.94" y2="71.12" width="0.4064" layer="16"/>
+<via x="27.94" y="71.12" extent="1-16" drill="0.6" shape="octagon"/>
+<wire x1="27.94" y1="83.82" x2="27.94" y2="86.36" width="0.4064" layer="16"/>
+<wire x1="27.94" y1="86.36" x2="26.67" y2="87.63" width="0.4064" layer="16"/>
 </signal>
 <signal name="S$15">
@@
 <wire x1="30.48" y1="91.44" x2="27.94" y2="91.44" width="0.4064" layer="16"/>
 </signal>
-<signal name="S$31">
-<contactref element="E$103" pad="2"/>
-<wire x1="27.94" y1="83.82" x2="27.94" y2="71.12" width="0.4064" layer="16"/>
-<via x="27.94" y="71.12" extent="1-16" drill="0.6" shape="octagon"/>
-</signal>
 <signal name="S$20">
